File: Order#100022604_2Layer_Green_1.6mm_HASL_5cm_x_5cm.sch (EAGLE design)
At the start: 22 parts, among them J2 GND +5V, T1 BC337, X1 22-23-2031, X2 22-23-2031, X3 22-23-2031, X5 22-23-2041

Commit message: Finito, paruo6ta siuntimui
Parts:
- removed J2: GND +5V, Connector:HEADER-2P-2.54
- added ETHERNET: ENC25J60, SparkFun-Connectors:M05X2PTH
- added IC1: REG1117, burr-brown:REG1117
- added J1: POWER, SparkFun-Connectors:POWER_JACKPTH_LOCK
- added JP4: (no value), SparkFun-Connectors:M03PTH
- added R10: 2k, resistor:R-EU_0207/10
- added R6: 3k3, resistor:R-EU_0207/10
- added R7: 1k, resistor:R-EU_0207/10
- added R8: 620, resistor:R-EU_0207/10
- added R9: 330, resistor:R-EU_0207/10
- added X4: GND A5 A4 VCC, con-molex:22-23-2041
- added X6: A6 A7, con-molex:22-23-2021
- JP1: value tx rx vcc gnd -> DTR TX RX VCC GDN
- JP3: value vcc tx rx gnd -> GND 3.3V; device SparkFun:ARDUINO_SERIAL_PROGRAMPTH -> SparkFun:M02PTH
- R2: value 4k7 -> 4k7
- S1: value (none) -> Right
- S2: value (none) -> Up
- S3: value (none) -> Down
- S4: value (none) -> Left
- S5: value (none) -> Select
- X1: value 22-23-2031 -> VCC D2 GND
- X2: value 22-23-2031 -> VCC D9 GND
- X3: value 22-23-2031 -> VCC A3 GND
- X5: value 22-23-2041 -> VCC A2 A1 GND
Connections:
- removed net N$3: R1.2
- removed net SCK: ARDUINO_PRO_MINI_2.9
- removed net VCC-TS: X1-3.S, X2-3.S, X3-3.S
- new net 3.3V: ETHERNET.9, IC1.VOUT, JP3.1
- new net A6: JP4.2, X6-1.S
- new net A7: JP4.1, X6-2.S
- new net D13: ARDUINO_PRO_MINI_2.9, ETHERNET.6
- new net N$11: R8.2, R9.1, S2.S, S2.S1
- new net N$5: R6.1, S5.S, S5.S1
- new net N$6: R6.2, R7.1, S4.S, S4.S1
- new net N$8: R7.2, R8.1, S3.S, S3.S1
- net A0: now also R10.1, R9.2, S1.S, S1.S1
- net A3: now also R2.2, X3-2.S
- net A4: now also X4-2.S
- net A5: now also LCD1602.4, X4-1.S
- net D10: now also ETHERNET.7; no longer R4.2, X3-2.S
- net D11: now also ETHERNET.5
- net D12: now also ETHERNET.4
- net D2: now also R4.2, X1-2.S; no longer LCD1602.4
- net D8: now also R1.2; no longer R2.2, X1-2.S
- net GND: now also ETHERNET.10, IC1.GND, J1.GND, J1.GNDBREAK, JP3.2, S1.P, S1.P1, S2.P, S2.P1, S3.P, S3.P1, S4.P, S4.P1, S5.P, S5.P1, X4-4.S; no longer J2.2, JP3.CTS
- net N$2: no longer LCD1602.2
- net RESET: now also ETHERNET.8
- net RXI: no longer JP3.TXO
- net TXO: no longer JP3.VCC
- net VCC: now also IC1.VIN, J1.PWR, LCD1602.2, R10.2, X1-3.S, X2-3.S, X3-3.S, X4-3.S; no longer J2.1, JP3.RXI
Other:
- moved on the sheet: R2, R4, S1, S2, S3, S4, S5
