File: solar_collector_controller_V2.brd (EAGLE design)
At the start: 49.5 x 50 mm, 29 parts, among them IC1 REG1117, J1 POWER_JACKSLT, T1 BC337, X1 22-23-2031, X2 22-23-2031, X3 22-23-2031, X5 22-23-2041

Commit message: pabaigta
Parts:
- added X4: VCC A4 A5 GND, con-molex:22-23-2041
- added X6: A7 A6, con-molex:22-23-2021
- ETHERNET: value M05X2PTH -> ENC25J60
- JP1: value tx rx vcc gnd -> DTR TX RX VCC GDN
- R2: value 4k7 -> 4k7
- X1: value 22-23-2031 -> GND D2 VCC
- X2: value 22-23-2031 -> GND D9 VCC
- X3: value 22-23-2031 -> GND A3 VCC
- X5: value 22-23-2041 -> GND A1 A2 VCC
- moved R1 25.7 mm to (11.4, 11.4), turned to 270 degrees
- moved R5 20.1 mm to (25.4, 38.1), turned to 0 degrees
- moved R2 2.84 mm to (14.0, 11.4)
- moved R3 2.84 mm to (16.5, 11.4)
- moved R4 2.84 mm to (19.1, 11.4)
- moved X1 2.54 mm to (29.2, 47.0)
- moved X2 2.54 mm to (19.1, 47.0)
- moved X3 2.54 mm to (8.89, 47.0)
- moved X5 2.54 mm to (40.6, 47.0)
- moved IC1 1.80 mm to (34.3, 39.4)
- moved ETHERNET 1.27 mm to (15.2, 40.6)
- moved R8 1.27 mm to (26.7, 26.7)
- turned T1 to 180 degrees
Connections:
- new net A6: JP4.2, X6.1
- new net A7: JP4.1, X6.2
- net A3: now also R2.2, X3.2
- net A4: now also X4.3; no longer R2.2, X1.2
- net A5: now also X4.2
- net D2: now also X1.2; no longer X3.2
- net GND: now also J1.GND@1, J1.GND@2, X4.1
- net VCC: now also J1.PWR, X4.4
Routing:
- net GND: track 0.00 -> 211.5 mm, vias 0 -> 2
- net VCC: track 0.00 -> 171.7 mm, vias 0 -> 1
- net D9: track 0.00 -> 92.5 mm, vias 0 -> 4
- net D10: track 0.00 -> 86.5 mm, vias 0 -> 2
- net D2: track 0.00 -> 67.5 mm, vias 0 -> 3
- net A1: track 0.00 -> 60.8 mm, vias 0 -> 3
- net A2: track 0.00 -> 58.6 mm, vias 0 -> 1
- net A5: track 0.00 -> 57.4 mm, vias 0 -> 3
- net D12: track 0.00 -> 49.0 mm, vias 0 -> 5
- net A3: track 0.00 -> 42.9 mm, vias 0 -> 4
- net D11: track 0.00 -> 40.0 mm, vias 0 -> 3
- net LCD16: track 0.00 -> 37.1 mm, vias 0 -> 1
- net D13: track 0.00 -> 37.0 mm, vias 0 -> 1
- net A7: track 0.00 -> 36.3 mm, vias 0 -> 1
- net N$8: track 0.00 -> 35.5 mm, vias 0 -> 1
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Other:
- board text added: "www.SauleVire.lt Saules kolektoriaus valdiklis V1.2 www.SauleVire.lt/en Solar collector controller V1.2"

Commit message: pastumdyta detalės...
Parts:
- added JP3: (no value), SparkFun:1X02
- J1: value POWER_JACKSLT -> POWER; device SparkFun-Connectors:POWER_JACK_SLOT -> SparkFun-Connectors:POWER_JACK_PTH_LOCK
- moved J1 28.6 mm to (52.7, 4.45)
- moved ETHERNET 27.5 mm to (27.3, 15.9), turned to 180 degrees
- moved IC1 25.1 mm to (38.1, 14.6)
- moved R10 22.9 mm to (26.0, 29.2), turned to 90 degrees
- moved X6 19.9 mm to (28.6, 2.54), turned to 180 degrees
- moved R9 16.4 mm to (22.2, 41.3), turned to 180 degrees
- moved R5 15.6 mm to (10.2, 41.3), turned to 270 degrees
- moved R6 15.3 mm to (31.8, 21.6)
- moved S2 14.7 mm to (31.8, 31.1)
- moved S1 14.6 mm to (37.5, 40.0)
- moved S4 14.6 mm to (38.7, 31.1)
- moved S5 14.6 mm to (38.1, 22.2)
- moved S3 14.6 mm to (45.7, 31.1)
- moved R7 12.9 mm to (22.2, 38.7), turned to 180 degrees
- moved X4 12.7 mm to (47.0, 15.2)
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Connections:
- net 3.3V: now also JP3.1
- net A4: now also X4.2; no longer X4.3
- net A5: now also X4.1; no longer X4.2
- net GND: now also J1.GND, J1.GNDBREAK, JP3.2, X4.4; no longer J1.GND@1, J1.GND@2, X4.1
- net VCC: now also X4.3; no longer X4.4
Routing:
- net D10: track 86.5 -> 19.2 mm, vias 2 -> 0
- net D12: track 49.0 -> 7.03 mm, vias 5 -> 0
- net D9: track 92.5 -> 55.6 mm, vias 4 -> 1
- net A0: track 26.9 -> 59.1 mm
- net D13: track 37.0 -> 7.03 mm, vias 1 -> 0
- net D11: track 40.0 -> 13.2 mm, vias 3 -> 0
- net A7: track 36.3 -> 13.1 mm, vias 1 -> 0
- net N$1: track 30.1 -> 8.18 mm
- net A6: track 33.8 -> 13.5 mm
- net A1: track 60.8 -> 43.9 mm, vias 3 -> 1
- net A2: track 58.6 -> 42.5 mm
- net 3.3V: track 10.8 -> 23.2 mm
- net RESET: track 32.8 -> 23.5 mm
- net GND: track 211.5 -> 204.2 mm, vias 2 -> 0
- net N$11: track 22.6 -> 15.5 mm
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
Commit message: padaryta
Parts:
- S1: value (none) -> Right
- S2: value (none) -> Up
- S3: value (none) -> Down
- S4: value (none) -> Left
- S5: value (none) -> Select
- moved S2 14.0 mm to (45.7, 31.1)
- moved S3 14.0 mm to (31.8, 31.1)
- moved R7 10.5 mm to (26.7, 29.2), turned to 90 degrees
- moved S5 8.91 mm to (38.7, 31.1), turned to 270 degrees
- moved S4 8.25 mm to (38.7, 22.9), turned to 180 degrees
- moved R10 7.96 mm to (22.2, 36.2), turned to 180 degrees
- moved R8 5.08 mm to (22.2, 41.3), turned to 180 degrees
- moved R9 2.54 mm to (22.2, 38.7), turned to 0 degrees
- moved S1 1.42 mm to (38.7, 39.4)
Routing:
- net N$11: track 15.5 -> 38.6 mm
- net N$8: track 37.2 -> 16.8 mm, vias 1 -> 0
- net A0: track 59.1 -> 43.2 mm
- net VCC: track 169.3 -> 155.7 mm
- net N$5: track 11.2 -> 23.2 mm, vias 0 -> 1
- net N$6: track 29.4 -> 19.9 mm, vias 0 -> 1
- net N$4: track 21.0 -> 27.1 mm
- net LCD16: track 38.3 -> 33.2 mm
- net GND: track 204.2 -> 199.1 mm
- net A4: track 32.9 -> 28.2 mm, vias 1 -> 0
- net A3: track 47.8 -> 43.9 mm, vias 1 -> 0
- net D2: track 67.5 -> 71.3 mm, vias 1 -> 0
- net D7: track 6.41 -> 10.2 mm
- net D9: track 55.6 -> 52.2 mm, vias 1 -> 0
- net A1: track 43.9 -> 40.9 mm
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Other:
- board text added: "ORDER #100022604"

Commit message: Finito, paruo6ta siuntimui
Parts:
- JP3: value (none) -> GND 3.3V
- X1: value GND D2 VCC -> VCC D2 GND
- X2: value GND D9 VCC -> VCC D9 GND
- X3: value GND A3 VCC -> VCC A3 GND
- X4: value VCC A4 A5 GND -> GND A5 A4 VCC
- X5: value GND A1 A2 VCC -> VCC A2 A1 GND
- X6: value A7 A6 -> A6 A7
Changed lines of the file:
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@@
 <element name="LCD1602" library="Connector_seedstudio" package="16P-2.54" value="" x="2.54" y="43.815" rot="R270"/>
 <element name="R5" library="resistor" package="RTRIM64W" value="10k" x="10.16" y="41.275" rot="R270"/>
-<element name="X1" library="con-molex" package="22-23-2031" value="GND D2 VCC" x="29.21" y="46.99" smashed="yes">
+<element name="X1" library="con-molex" package="22-23-2031" value="VCC D2 GND" x="29.21" y="46.99" smashed="yes">
 <attribute name="OC_NEWARK" value="30C0862" x="29.21" y="46.99" size="1.778" layer="27" display="off"/>
 <attribute name="MPN" value="22-23-2031" x="29.21" y="46.99" size="1.778" layer="27" display="off"/>
@@
 <attribute name="OC_FARNELL" value="1462950" x="29.21" y="46.99" size="1.778" layer="27" display="off"/>
 <attribute name="NAME" x="25.4" y="50.8" size="1.016" layer="25" ratio="10"/>
-<attribute name="VALUE" x="26.035" y="48.895" size="0.8" layer="27" ratio="10"/>
+<attribute name="VALUE" x="32.385" y="48.895" size="0.8" layer="28" ratio="10" rot="MR0"/>
 </element>
-<element name="X2" library="con-molex" package="22-23-2031" value="GND D9 VCC" x="19.05" y="46.99" smashed="yes">
+<element name="X2" library="con-molex" package="22-23-2031" value="VCC D9 GND" x="19.05" y="46.99" smashed="yes">
 <attribute name="OC_NEWARK" value="30C0862" x="19.05" y="46.99" size="1.778" layer="27" display="off"/>
 <attribute name="MPN" value="22-23-2031" x="19.05" y="46.99" size="1.778" layer="27" display="off"/>
@@
 <attribute name="OC_FARNELL" value="1462950" x="19.05" y="46.99" size="1.778" layer="27" display="off"/>
 <attribute name="NAME" x="15.24" y="50.8" size="1.016" layer="25" ratio="10"/>
-<attribute name="VALUE" x="15.875" y="48.895" size="0.8" layer="27" ratio="10"/>
+<attribute name="VALUE" x="22.225" y="48.895" size="0.8" layer="28" ratio="10" rot="MR0"/>
 </element>
-<element name="X3" library="con-molex" package="22-23-2031" value="GND A3 VCC" x="8.89" y="46.99" smashed="yes">
+<element name="X3" library="con-molex" package="22-23-2031" value="VCC A3 GND" x="8.89" y="46.99" smashed="yes">
 <attribute name="OC_NEWARK" value="30C0862" x="8.89" y="46.99" size="1.778" layer="27" display="off"/>
 <attribute name="MPN" value="22-23-2031" x="8.89" y="46.99" size="1.778" layer="27" display="off"/>
@@
 <attribute name="OC_FARNELL" value="1462950" x="8.89" y="46.99" size="1.778" layer="27" display="off"/>
 <attribute name="NAME" x="5.08" y="50.8" size="1.016" layer="25" ratio="10"/>
-<attribute name="VALUE" x="5.715" y="48.895" size="0.8" layer="27" ratio="10"/>
+<attribute name="VALUE" x="12.065" y="48.895" size="0.8" layer="28" ratio="10" rot="MR0"/>
 </element>
 <element name="S1" library="switch-omron" package="B3F-10XX" value="Right" x="38.735" y="39.37" smashed="yes" rot="R180">
@@
 <attribute name="OC_FARNELL" value="176432" x="38.735" y="31.115" size="1.778" layer="27" rot="R270" display="off"/>
 </element>
-<element name="X5" library="con-molex" package="22-23-2041" value="GND A1   A2 VCC" x="40.64" y="46.99" smashed="yes">
+<element name="X5" library="con-molex" package="22-23-2041" value="VCC A2   A1 GND" x="40.64" y="46.99" smashed="yes">
 <attribute name="OC_NEWARK" value="38C0355" x="40.64" y="46.99" size="1.778" layer="27" display="off"/>
 <attribute name="MPN" value="22-23-2041" x="40.64" y="46.99" size="1.778" layer="27" display="off"/>
@@
 <attribute name="OC_FARNELL" value="1462920" x="40.64" y="46.99" size="1.778" layer="27" display="off"/>
 <attribute name="NAME" x="35.56" y="50.8" size="1.016" layer="25" ratio="10"/>
-<attribute name="VALUE" x="36.195" y="48.895" size="0.8" layer="27" ratio="10"/>
+<attribute name="VALUE" x="36.195" y="49.53" size="0.8" layer="28" ratio="10" rot="MR180"/>
 </element>
 <element name="T1" library="transistor" package="TO92" value="BC337" x="6.35" y="36.83" smashed="yes" rot="R180">
 <attribute name="NAME" x="3.175" y="36.195" size="1.27" layer="25" ratio="10" rot="R180"/>
-<attribute name="VALUE" x="3.175" y="38.1" size="1.27" layer="27" ratio="10" rot="R180"/>
+<attribute name="VALUE" x="13.97" y="38.735" size="1.27" layer="27" ratio="10" rot="R180"/>
 </element>
 <element name="R6" library="resistor" package="0207/10" value="3k3" x="31.75" y="21.59" smashed="yes" rot="R90">
@@
 <attribute name="VALUE" x="33.528" y="18.034" size="1.27" layer="27" ratio="10" rot="R270"/>
 </element>
-<element name="X4" library="con-molex" package="22-23-2041" value="VCC A4 A5 GND" x="46.99" y="15.24" smashed="yes" rot="R270">
+<element name="X4" library="con-molex" package="22-23-2041" value="GND A5 A4 VCC" x="46.99" y="15.24" smashed="yes" rot="R270">
 <attribute name="OC_NEWARK" value="38C0355" x="46.99" y="15.24" size="1.778" layer="27" rot="R270" display="off"/>
 <attribute name="MPN" value="22-23-2041" x="46.99" y="15.24" size="1.778" layer="27" rot="R270" display="off"/>
@@
 <attribute name="OC_FARNELL" value="1462920" x="46.99" y="15.24" size="1.778" layer="27" rot="R270" display="off"/>
 <attribute name="NAME" x="48.895" y="14.605" size="1.016" layer="25" ratio="10" rot="R270"/>
-<attribute name="VALUE" x="46.99" y="20.32" size="1.016" layer="27" ratio="10" rot="R270"/>
+<attribute name="VALUE" x="46.99" y="20.32" size="1.016" layer="28" ratio="10" rot="MR270"/>
 </element>
-<element name="X6" library="con-molex" package="22-23-2021" value="   A7 A6" x="28.575" y="2.54" smashed="yes" rot="R180">
+<element name="X6" library="con-molex" package="22-23-2021" value="   A6 A7" x="28.575" y="2.54" smashed="yes" rot="R180">
 <attribute name="OC_NEWARK" value="25C3832" x="28.575" y="2.54" size="1.778" layer="27" rot="R180" display="off"/>
 <attribute name="MPN" value="22-23-2021" x="28.575" y="2.54" size="1.778" layer="27" rot="R180" display="off"/>
@@
 <attribute name="OC_FARNELL" value="1462926" x="28.575" y="2.54" size="1.778" layer="27" rot="R180" display="off"/>
 <attribute name="NAME" x="31.115" y="-1.27" size="1.016" layer="25" ratio="10" rot="R180"/>
-<attribute name="VALUE" x="30.48" y="5.08" size="1.016" layer="27" ratio="10" rot="R180"/>
+<attribute name="VALUE" x="26.67" y="5.08" size="1.016" layer="28" ratio="10" rot="MR180"/>
 </element>
-<element name="JP3" library="SparkFun" package="1X02" value="" x="33.02" y="1.905"/>
+<element name="JP3" library="SparkFun" package="1X02" value="GND 3.3V" x="33.02" y="1.905" smashed="yes">
+<attribute name="NAME" x="32.9438" y="-0.0762" size="1.27" layer="25" ratio="10"/>
+<attribute name="VALUE" x="37.465" y="3.175" size="1" layer="28" rot="MR0"/>
+</element>
 </elements>
 <signals>
