File: solar_collector_controller_V2.sch (EAGLE design)
At the start: 28 parts, among them J2 GND +5V, T1 BC337, X1 22-23-2031, X2 22-23-2031, X3 22-23-2031, X5 22-23-2041

Commit message: pridetas tinklas, 3.3v
Parts:
- removed DIS1: TUXGR_16X2_R2, display-lcd:TUXGR_16X2_R2
- removed J2: GND +5V, Connector:HEADER-2P-2.54
- removed JP3: vcc tx rx gnd, SparkFun:ARDUINO_SERIAL_PROGRAMPTH
- added ETHERNET: M05X2PTH, SparkFun-Connectors:M05X2PTH
- added IC1: REG1117, burr-brown:REG1117
- added J1: POWER_JACKSLT, SparkFun-Connectors:POWER_JACKSLT
- added JP4: (no value), SparkFun-Connectors:M03PTH
Connections:
- removed net N$13: R10.1, R9.2, S1.S, S1.S1
- removed net N$3: R1.2
- removed net SCK: ARDUINO_PRO_MINI_2.9
- new net 3.3V: ETHERNET.9, IC1.VOUT
- new net D13: ARDUINO_PRO_MINI_2.9, ETHERNET.6
- net A0: now also R10.1, R9.2, S1.S, S1.S1
- net A4: now also R2.2, X1-2.S
- net A5: now also LCD1602.4
- net D10: now also R1.2; no longer R4.2, X3-2.S
- net D11: now also ETHERNET.5
- net D12: now also ETHERNET.4
- net D2: now also ETHERNET.2; no longer LCD1602.4
- net D8: now also ETHERNET.7; no longer R2.2, X1-2.S
- net GND: now also ETHERNET.10, IC1.GND; no longer J2.2, JP3.CTS
- net N$2: no longer LCD1602.2
- net RESET: now also ETHERNET.8
- net RXI: no longer JP3.TXO
- net TXO: no longer JP3.VCC
- net VCC: now also IC1.VIN, LCD1602.2; no longer J2.1, JP3.RXI
Other:
- moved on the sheet: R2

Commit message: i6mestas pertraukimas
Connections:
- removed net VCC-TS: X1-3.S, X2-3.S, X3-3.S
- net D10: now also ETHERNET.7; no longer R1.2
- net D2: now also R4.2, X3-2.S; no longer ETHERNET.2
- net D8: now also R1.2; no longer ETHERNET.7
- net VCC: now also X1-3.S, X2-3.S, X3-3.S
Other:
- moved on the sheet: R4
Changed lines of the file:
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@@
 <instance part="R2" gate="G$1" x="93.98" y="83.82"/>
 <instance part="R3" gate="G$1" x="86.36" y="91.44" rot="R90"/>
-<instance part="R4" gate="G$1" x="149.86" y="88.9" rot="R90"/>
+<instance part="R4" gate="G$1" x="78.74" y="109.22" rot="R90"/>
 <instance part="LCD1602" gate="G$1" x="55.88" y="106.68"/>
 <instance part="R5" gate="G$1" x="78.74" y="83.82" rot="R90"/>
@@
 <label x="88.9" y="114.3" size="1.778" layer="95" rot="MR0"/>
 <pinref part="ARDUINO_PRO_MINI_1" gate="G$1" pin="8"/>
-</segment>
-<segment>
-<pinref part="ETHERNET" gate="G$1" pin="2"/>
-<wire x1="172.72" y1="66.04" x2="180.34" y2="66.04" width="0.1524" layer="91"/>
-<label x="175.26" y="66.04" size="1.778" layer="95"/>
+<pinref part="R4" gate="G$1" pin="2"/>
+<wire x1="83.82" y1="114.3" x2="78.74" y2="114.3" width="0.1524" layer="91"/>
+</segment>
+<segment>
+<pinref part="X3" gate="-2" pin="S"/>
+<wire x1="175.26" y1="96.52" x2="170.18" y2="96.52" width="0.1524" layer="91"/>
+<label x="170.18" y="96.52" size="1.778" layer="95"/>
 </segment>
 </net>
@@
 </segment>
 <segment>
-<pinref part="R1" gate="G$1" pin="2"/>
-<wire x1="63.5" y1="53.34" x2="63.5" y2="60.96" width="0.1524" layer="91"/>
-<label x="63.5" y="58.42" size="1.778" layer="95"/>
+<pinref part="ETHERNET" gate="G$1" pin="7"/>
+<wire x1="157.48" y1="58.42" x2="149.86" y2="58.42" width="0.1524" layer="91"/>
+<label x="149.86" y="58.42" size="1.778" layer="95"/>
 </segment>
 </net>
@@
 <wire x1="157.48" y1="60.96" x2="149.86" y2="60.96" width="0.1524" layer="91"/>
 <label x="149.86" y="60.96" size="1.778" layer="95"/>
-</segment>
-</net>
-<net name="VCC-TS" class="0">
-<segment>
-<pinref part="X2" gate="-3" pin="S"/>
-<wire x1="175.26" y1="106.68" x2="170.18" y2="106.68" width="0.1524" layer="91"/>
-<label x="167.64" y="106.68" size="1.778" layer="95"/>
-</segment>
-<segment>
-<pinref part="X3" gate="-3" pin="S"/>
-<wire x1="175.26" y1="93.98" x2="170.18" y2="93.98" width="0.1524" layer="91"/>
-<label x="182.88" y="106.68" size="1.778" layer="95"/>
-</segment>
-<segment>
-<pinref part="X1" gate="-3" pin="S"/>
-<wire x1="175.26" y1="121.92" x2="170.18" y2="121.92" width="0.1524" layer="91"/>
-<label x="167.64" y="121.92" size="1.778" layer="95"/>
 </segment>
 </net>
@@
 <segment>
 <pinref part="R4" gate="G$1" pin="1"/>
-<wire x1="149.86" y1="83.82" x2="149.86" y2="78.74" width="0.1524" layer="91"/>
-<label x="149.86" y="81.28" size="1.778" layer="95"/>
+<wire x1="78.74" y1="104.14" x2="78.74" y2="99.06" width="0.1524" layer="91"/>
+<label x="76.2" y="99.06" size="1.778" layer="95"/>
 </segment>
 <segment>
@@
 <wire x1="66.04" y1="88.9" x2="71.12" y2="88.9" width="0.1524" layer="91"/>
 <label x="66.04" y="88.9" size="1.778" layer="95"/>
+</segment>
+<segment>
+<pinref part="X3" gate="-3" pin="S"/>
+<wire x1="175.26" y1="93.98" x2="170.18" y2="93.98" width="0.1524" layer="91"/>
+<label x="170.18" y="93.98" size="1.778" layer="95"/>
+</segment>
+<segment>
+<pinref part="X2" gate="-3" pin="S"/>
+<wire x1="175.26" y1="106.68" x2="170.18" y2="106.68" width="0.1524" layer="91"/>
+<label x="167.64" y="106.68" size="1.778" layer="95"/>
+</segment>
+<segment>
+<pinref part="X1" gate="-3" pin="S"/>
+<wire x1="175.26" y1="121.92" x2="170.18" y2="121.92" width="0.1524" layer="91"/>
+<label x="167.64" y="121.92" size="1.778" layer="95"/>
 </segment>
 </net>
@@
 </segment>
 <segment>
-<pinref part="ETHERNET" gate="G$1" pin="7"/>
-<wire x1="157.48" y1="58.42" x2="149.86" y2="58.42" width="0.1524" layer="91"/>
-<label x="149.86" y="58.42" size="1.778" layer="95"/>
-</segment>
-</net>
+<pinref part="R1" gate="G$1" pin="2"/>
+<wire x1="63.5" y1="53.34" x2="63.5" y2="60.96" width="0.1524" layer="91"/>
+<label x="63.5" y="58.42" size="1.778" layer="95"/>
+</segment>
+</net>

Commit message: pabaigta
Parts:
- added X4: VCC A4 A5 GND, con-molex:22-23-2041
- added X6: A7 A6, con-molex:22-23-2021
- ETHERNET: value M05X2PTH -> ENC25J60
- JP1: value tx rx vcc gnd -> DTR TX RX VCC GDN
- R2: value 4k7 -> 4k7
- X1: value 22-23-2031 -> GND D2 VCC
- X2: value 22-23-2031 -> GND D9 VCC
- X3: value 22-23-2031 -> GND A3 VCC
- X5: value 22-23-2041 -> GND A1 A2 VCC
Connections:
- new net A6: JP4.2, X6-1.S
- new net A7: JP4.1, X6-2.S
- net A3: now also R2.2, X3-2.S
- net A4: now also X4-3.S; no longer R2.2, X1-2.S
- net A5: now also X4-2.S
- net D2: now also X1-2.S; no longer X3-2.S
- net GND: now also J1.GND, J1.GNDBREAK, X4-1.S
- net VCC: now also J1.PWR, X4-4.S
Other:
- moved on the sheet: JP4

Commit message: pastumdyta detalės...
Parts:
- added JP3: (no value), SparkFun:M02PTH
- J1: value POWER_JACKSLT -> POWER; device SparkFun-Connectors:POWER_JACKSLT -> SparkFun-Connectors:POWER_JACKPTH_LOCK
Connections:
- net 3.3V: now also JP3.1
- net A4: now also X4-2.S; no longer X4-3.S
- net A5: now also X4-1.S; no longer X4-2.S
- net GND: now also JP3.2, X4-4.S; no longer X4-1.S
- net VCC: now also X4-3.S; no longer X4-4.S

Commit message: padaryta
Parts:
- S1: value (none) -> Right
- S2: value (none) -> Up
- S3: value (none) -> Down
- S4: value (none) -> Left
- S5: value (none) -> Select
Changed lines of the file:
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@@
 <part name="X2" library="con-molex" deviceset="22-23-2031" device="" value="GND D9 VCC"/>
 <part name="X3" library="con-molex" deviceset="22-23-2031" device="" value="GND A3 VCC"/>
-<part name="S1" library="switch-omron" deviceset="10-XX" device=""/>
-<part name="S2" library="switch-omron" deviceset="10-XX" device=""/>
-<part name="S3" library="switch-omron" deviceset="10-XX" device=""/>
-<part name="S4" library="switch-omron" deviceset="10-XX" device=""/>
-<part name="S5" library="switch-omron" deviceset="10-XX" device=""/>
+<part name="S1" library="switch-omron" deviceset="10-XX" device="" value="Right"/>
+<part name="S2" library="switch-omron" deviceset="10-XX" device="" value="Up"/>
+<part name="S3" library="switch-omron" deviceset="10-XX" device="" value="Down"/>
+<part name="S4" library="switch-omron" deviceset="10-XX" device="" value="Left"/>
+<part name="S5" library="switch-omron" deviceset="10-XX" device="" value="Select"/>
 <part name="X5" library="con-molex" deviceset="22-23-2041" device="" value="GND A1   A2 VCC"/>
 <part name="T1" library="transistor" deviceset="BC337" device=""/>
@@
 <instance part="X3" gate="-2" x="177.8" y="96.52"/>
 <instance part="X3" gate="-3" x="177.8" y="93.98"/>
-<instance part="S1" gate="1" x="208.28" y="121.92" rot="R270"/>
-<instance part="S2" gate="1" x="208.28" y="109.22" rot="R270"/>
-<instance part="S3" gate="1" x="208.28" y="96.52" rot="R270"/>
-<instance part="S4" gate="1" x="208.28" y="83.82" rot="R270"/>
-<instance part="S5" gate="1" x="208.28" y="71.12" rot="R270"/>
+<instance part="S1" gate="1" x="208.28" y="121.92" smashed="yes" rot="R270">
+<attribute name="NAME" x="205.74" y="128.27" size="1.778" layer="95"/>
+<attribute name="VALUE" x="196.215" y="120.65" size="1.778" layer="96"/>
+</instance>
+<instance part="S2" gate="1" x="208.28" y="109.22" smashed="yes" rot="R270">
+<attribute name="NAME" x="205.74" y="115.57" size="1.778" layer="95"/>
+<attribute name="VALUE" x="198.755" y="107.95" size="1.778" layer="96"/>
+</instance>
+<instance part="S3" gate="1" x="208.28" y="96.52" smashed="yes" rot="R270">
+<attribute name="NAME" x="205.74" y="102.87" size="1.778" layer="95"/>
+<attribute name="VALUE" x="193.675" y="95.25" size="1.778" layer="96"/>
+</instance>
+<instance part="S4" gate="1" x="208.28" y="83.82" smashed="yes" rot="R270">
+<attribute name="NAME" x="205.74" y="90.17" size="1.778" layer="95"/>
+<attribute name="VALUE" x="193.675" y="82.55" size="1.778" layer="96"/>
+</instance>
+<instance part="S5" gate="1" x="208.28" y="71.12" smashed="yes" rot="R270">
+<attribute name="NAME" x="205.74" y="77.47" size="1.778" layer="95"/>
+<attribute name="VALUE" x="193.675" y="72.39" size="1.778" layer="96"/>
+</instance>
 <instance part="X5" gate="-1" x="93.98" y="55.88"/>
 <instance part="X5" gate="-2" x="93.98" y="53.34"/>

Commit message: Finito, paruo6ta siuntimui
Parts:
- JP3: value (none) -> GND 3.3V
- X1: value GND D2 VCC -> VCC D2 GND
- X2: value GND D9 VCC -> VCC D9 GND
- X3: value GND A3 VCC -> VCC A3 GND
- X4: value VCC A4 A5 GND -> GND A5 A4 VCC
- X5: value GND A1 A2 VCC -> VCC A2 A1 GND
- X6: value A7 A6 -> A6 A7
Changed lines of the file:
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@@
 <part name="LCD1602" library="Connector_seedstudio" deviceset="HEADER-16P" device="-2.54"/>
 <part name="R5" library="resistor" deviceset="R-TRIMM" device="64W" value="10k"/>
-<part name="X1" library="con-molex" deviceset="22-23-2031" device="" value="GND D2 VCC"/>
-<part name="X2" library="con-molex" deviceset="22-23-2031" device="" value="GND D9 VCC"/>
-<part name="X3" library="con-molex" deviceset="22-23-2031" device="" value="GND A3 VCC"/>
+<part name="X1" library="con-molex" deviceset="22-23-2031" device="" value="VCC D2 GND"/>
+<part name="X2" library="con-molex" deviceset="22-23-2031" device="" value="VCC D9 GND"/>
+<part name="X3" library="con-molex" deviceset="22-23-2031" device="" value="VCC A3 GND"/>
 <part name="S1" library="switch-omron" deviceset="10-XX" device="" value="Right"/>
 <part name="S2" library="switch-omron" deviceset="10-XX" device="" value="Up"/>
@@
 <part name="S4" library="switch-omron" deviceset="10-XX" device="" value="Left"/>
 <part name="S5" library="switch-omron" deviceset="10-XX" device="" value="Select"/>
-<part name="X5" library="con-molex" deviceset="22-23-2041" device="" value="GND A1   A2 VCC"/>
+<part name="X5" library="con-molex" deviceset="22-23-2041" device="" value="VCC A2   A1 GND"/>
 <part name="T1" library="transistor" deviceset="BC337" device=""/>
 <part name="R6" library="resistor" deviceset="R-EU_" device="0207/10" value="3k3"/>
@@
 <part name="J1" library="SparkFun-Connectors" deviceset="POWER_JACK" device="PTH_LOCK" value="POWER"/>
 <part name="IC1" library="burr-brown" deviceset="REG1117" device=""/>
-<part name="X4" library="con-molex" deviceset="22-23-2041" device="" value="VCC A4 A5 GND"/>
-<part name="X6" library="con-molex" deviceset="22-23-2021" device="" value="   A7 A6"/>
-<part name="JP3" library="SparkFun" deviceset="M02" device="PTH"/>
+<part name="X4" library="con-molex" deviceset="22-23-2041" device="" value="GND A5 A4 VCC"/>
+<part name="X6" library="con-molex" deviceset="22-23-2021" device="" value="   A6 A7"/>
+<part name="JP3" library="SparkFun" deviceset="M02" device="PTH" value="GND 3.3V"/>
 </parts>
 <sheets>
@@
 <pinref part="JP3" gate="G$1" pin="2"/>
 <wire x1="109.22" y1="38.1" x2="104.14" y2="38.1" width="0.1524" layer="91"/>
+<label x="104.14" y="38.1" size="1.778" layer="95"/>
 </segment>
 </net>
@@
 <pinref part="JP3" gate="G$1" pin="1"/>
 <wire x1="109.22" y1="40.64" x2="104.14" y2="40.64" width="0.1524" layer="91"/>
-</segment>
-</net>
+<label x="104.14" y="40.64" size="1.778" layer="95"/>
+</segment>
+</net>
