File: os20.oldenc.sch (EAGLE design)
At the start: 82 parts, among them IC2 LM1117-33, IC6 ENC28J60, K1 G5V1, K2 G5V1, K3 G5V1, T1 2N2222, T2 2N2222, T3 2N2222, T4 2N2222, U1 ATMEGA328P, X1 25MHz, X2 32.768kHz, X3 25MHz, X7 22-23-2031, X8 22-23-2031, X9 22-23-2031

Commit message: pcb
prie pabaigos...
Parts:
- removed DOWN, LEFT, RESET, RIGHT, SELECT, UP: (no value), SparkFun-Electromechanical:TAC_SWITCHPTH
- removed K1, K2, K3: G5V1, relay:G5V1
- removed LED1, LED2, LED3: (no value), adafruit:LEDSMT1206
- removed R1, R10: 1k, rcl:R-EU_R0805
- removed R11: 620, rcl:R-EU_R0805
- removed R12: 330, rcl:R-EU_R0805
- removed R13: 2k, rcl:R-EU_R0805
- removed R14, R17, R25, R9: 3k3, rcl:R-EU_R0805
- removed R15, R18, R26: 470, rcl:R-EU_R0805
- removed R16, R2, R23, R24, R3, R4, R5, R6: 10k, rcl:R-EU_R0805
- removed R19, R20, R21, R22: 49, rcl:R-EU_R0805
- removed R7, R8: 47, rcl:R-EU_R0805
- removed U$1: FRAME_DINA4_L, dp_devices:FRAME_DINA4_L
- removed U$2: CELLPHONE_NOKIA_5100, DIY-Cellphone:CELLPHONE_NOKIA_5100
- removed X10, X12, X13: (no value), con-phoenix-254:MPT3
- removed X11: (no value), con-phoenix-254:MPT2
- removed X3: 25MHz, SparkFun:CRYSTALHC49US
- removed X7, X8, X9: 22-23-2031, con-molex:22-23-2031
- added B1, B2, B3: (no value), adafruit:31-XX
- added C1': 100u, resistor:CPOL-EUE
- added COM, RAIN, S12, S34, S56, S78: (no value), SparkFun:M025MM
- added CX1, CX2: 18p, resistor:C-EUC0805
- added DF1, DF2, DF3, DF4, DF5, DF6, DF7, DF8: (no value), diode:DIODE-D-2.5
- added EXTOUT: (no value), pinhead:PINHD-2X4
- added F1: 1A, adafruit:PTCFUSE-1812
- added IC1: LM2596S-5.0, national-semiconductor:LM2596S
- added IC5: 74HC595N, SparkFun:74LS595D
- added IC8: ATMEGA644A, atmel:ATMEGA644A
- added J0: 24VAC IN, SparkFun:M025MM
- added J2: EG1206, adafruit:EG1206
- added JP2, JP3, JP4, JP5, JP6, JP7, JP8, JP9, P1, P2: (no value), adafruit:PINHD-1X1CB
- added L1: 150uH, rcl:L-US6000-XXX-RC
- added L1': 220uH, SparkFunNew:INDUCTORPWR
- added LCD: HD44780LCDNOHOLE, adafruit:HD44780LCDNOHOLE
- added P0: (no value), adafruit:PINHD-1X14-CB
- added P4, P5: (no value), pinhead:PINHD-1X3
- added R+, R-: 47, rcl:R-EU_R0805
- added RN1, RN2, RN3: (no value), resistor-dil:4R-NEXB38V
- added RN4: 49.9, resistor-dil:4R-NEXB38V
- added RPR: 1.5K, rcl:R-EU_R0805
- added T5, T6, T7, T8: MAC97, SparkFun:MAC97SOT223
- added V1, V2, V3, V4, V5, V6, V7, V8: MOV, varistor:VARISTOR-5
- added X1'1: 32.657k, crystal:CRYSTALMM20SS
- added X2': 25MHz, SparkFun:CRYSTALHC49US
- C1: value 18p -> 100u; device resistor:C-EUC0805 -> resistor:CPOL-EUE3.5-8
- C2: value 18p -> 100u; device resistor:C-EUC0805 -> resistor:CPOL-EUD
- C4, C5: value 22p -> 0.1u; device resistor:C-EUC0805 -> rcl:C-EUC0805
- C6: value 100n -> 0.1u; device resistor:C-EUC0805 -> rcl:C-EUC0805
- D1: value (none) -> S1A; device adafruit:DIODEDO-1N4148 -> diode:DIODE-DO-214AC
- D2: value (none) -> 5.1V; device adafruit:DIODEDO-1N4148 -> diode:DIODE-MINIMELF
- D3: value (none) -> SS24; device adafruit:DIODEDO-1N4148 -> diode:DIODE-DO-214AC
- IC6: device SparkFun-DigitalIC:ENC28J60 -> SparkFun:ENC28J60SO28LONG
- T1, T2, T3, T4: value 2N2222 -> MAC97; device adafruit:2N2222 -> SparkFun:MAC97SOT223
- U1: value ATMEGA328P -> USD-SOCKETMICRO-SD-SOCKET-TAOBAO; device SparkFun-DigitalIC:ATMEGA328_SMT -> SparkFunNew:USD-SOCKETMICRO-SD-SOCKET-TAOBAO
- USB: value (none) -> USBPTH; device adafruit:USBMOLEX -> SparkFunNew:USBPTH
- X1: value 25MHz -> 32.657k; device SparkFun:CRYSTALHC49US -> crystal:CRYSTALTC26H
- X2: value 32.768kHz -> 25MHz; device crystal:CRYSTALTC26H -> SparkFun:CRYSTAL10.5X4.8
- renumbered ATTINY to IC7, DS1307 to IC3, RJ45 to RJ1
Connections:
- removed net +3V3: C3.+, IC2.OUT@1, IC6.VDD, IC6.VDDOSC, IC6.VDDPLL, IC6.VDDRX, IC6.VDDTX
- removed net +5V: C9.1, D1.C, D2.C, D3.C, IC2.IN, IC3.VCC, IC7.VCC, K11.1, K21.1, K31.1, LED2.A, LED3.A, R23.2, R24.2, U$2.VCC, X10-3.1, X12-3.1, X13-3.1
- removed net D10: R1.2, U1.PB2(SS/OC1B)
- removed net D11: IC6.SI, U1.PB3(MOSI/OC2)
- removed net D2: U1.PD2(INT0), X13-2.1
- removed net D5: R4.2, U1.PD5(T1)
- removed net D6: R5.2, U1.PD6(AIN0)
- removed net D7: R6.2, U1.PD7(AIN1)
- removed net D8: IC6.CS, U1.PB0(ICP)
- removed net D9: U1.PB1(OC1A)
- removed net N$31: LED3.C, R26.1
- removed net N$32: C4.2, U1.PB7(XTAL2/TOSC2), X3.1
- removed net N$33: C5.2, U1.PB6(XTAL1/TOSC1), X3.2
- removed net N$35: C6.1, U1.AREF
- removed net N$44: R1.1, T4.B
- removed net N$46: R16.1, RESET.3, RESET.4, U1.PC6(/RESET)
- removed net V$: R6.1, U$2.RST
- new net 24VAC: COM.1, COM.2, D1.A, DF1.C, DF2.C, DF3.C, DF4.C, DF5.C, DF6.C, DF7.C, DF8.C, J2.S
- new net A4: EXTOUT.3, IC8.(PCINT4/ADC4)PA4, RPR.1
- new net A5: IC8.(PCINT5/ADC5)PA5, P0.9
- new net AREF: C5.1, IC8.AREF
- new net D14: IC8.(PCINT30/OC2B/ICP)PD6, P0.2
- new net D15: IC8.(PCINT31/OC2A)PD7, P0.1
- new net D18: IC8.(PCINT18/TCK)PC2, LCD.E
- new net D19: IC8.(PCINT19/TMS)PC3, LCD.RS
- new net D20: IC8.(PCINT20/TDO)PC4, LCD.DB4
- new net D21: IC5.SER, IC8.(PCINT21/TDI)PC5, LCD.DB5
- new net D22: EXTOUT.4, IC5.SCK, IC8.(PCINT22/TOSC1)PC6, LCD.DB6
- new net D23: IC8.(PCINT23/TOSC2)PC7, LCD.DB7
- new net INT0: IC8.(PCINT26/INT0)PD2, P0.4
- new net INT1: IC8.(PCINT27/INT1)PD3, RAIN.2
- new net INT2: IC8.(PCINT10/INT2/AIN0)PB2, P0.3
- new net N$10: IC5.QE, RN3A.2
- new net QH*: EXTOUT.2, IC5.QH*
- new net RXD: IC8.(PCINT24/RXD0)PD0, P0.6
- new net TXD: IC8.(PCINT25/TXD0)PD1, P0.5
- net A0: now also B1.P, IC8.(PCINT0/ADC0)PA0; no longer U1.PC0(ADC0)
- net A1: now also B2.P, IC8.(PCINT1/ADC1)PA1; no longer U1.PC1(ADC1), X12-2.1
- net A2: now also B3.P, IC8.(PCINT2/ADC2)PA2; no longer R17.2, U1.PC2(ADC2)
- net A3: now also IC8.(PCINT3/ADC3)PA3, P4.1, P5.2; no longer R14.2, U1.PC3(ADC3)
- net A6: now also IC8.(PCINT6/ADC6)PA6, P0.8; no longer R12.2, R13.1, RIGHT.3, RIGHT.4, U1.ADC6
- net A7: now also IC8.(PCINT7/ADC7)PA7, P0.7; no longer U1.ADC7
- net D+: now also R-.1; no longer R8.1
- net D-: now also R+.1; no longer R7.1
- net D0: now also IC8.(PCINT8/XCK0/T0)PB0, U1.CS; no longer R25.2, U1.PD0(RXD)
- net D1: now also EXTOUT.8, IC5.G, IC8.(PCINT9/CLKO/T1)PB1, RN1B.1; no longer U1.PD1(TXD), X10-2.1
- net D12: now also IC8.(PCINT28/OC1B)PD4, LCD.K; no longer IC6.SO, U1.PB4(MISO)
- net D13: now also IC8.(PCINT29/OC1A)PD5, LCD.VO; no longer IC6.SCK, U1.PB5(SCK)
- net D3: now also EXTOUT.6, IC5.RCK, IC8.(PCINT11/OC0A/AIN1)PB3; no longer R2.2, U1.PD3(INT1)
- net D4: now also IC6.CS, IC8.(PCINT12/OC0B/!SS!)PB4; no longer R3.2, U1.PD4(XCK/T0)
- net GND: now also B1.S, B2.S, B3.S, C1'.-, C1.-, C2.-, C4.2, C5.2, CX1.2, CX2.2, D2.A, D3.A, EXTOUT.5, EXTOUT.7, IC1.!ON!/OFF, IC1.GND, IC5.GND, IC8.GND, IC8.GND@1, IC8.GND@2, IC8.GND@3, J0.1, LCD.RW, LCD.VSS, P0.14, P2.1, P4.3, P5.3, RAIN.1, T1.M1, T2.M1, T3.M1, T4.M1, T5.M1, T6.M1, T7.M1, T8.M1, U1.GND, U1.SHIELD@1, U1.SHIELD@2, U1.SHIELD@3, U1.SHIELD@4, V1.1, V2.1, V3.1, V4.1, V5.1, V6.1, V7.1, V8.1; no longer C1.2, C2.2, C4.1, C5.1, DOWN.1, DOWN.2, LEFT.1, LEFT.2, RESET.1, RESET.2, RIGHT.1, SELECT.1, SELECT.2, T1.E, T2.E, T3.E, T4.E, U$2.GND, U1.AGND, U1.GND@1, U1.GND@2, UP.1, UP.2, USB.ID, X10-1.1, X12-1.1, X13-1.1
- net MISO: now also IC6.SO, IC8.(PCINT14/MISO)PB6, U1.DO
- net MOSI: now also IC6.SI, IC8.(PCINT13/MOSI)PB5, U1.DI
- net N$1: now also C1'.+, C1.+, D1.C, IC1.VIN; no longer LEFT.3, LEFT.4, R10.1, R9.2
- net N$11: now also IC5.QD, RN2D.2; no longer D3.A, K31.2, R26.2, T2.C
- net N$12: now also IC5.QC, RN2C.2; no longer D2.A, K11.2, R18.2, T3.C
- net N$13: now also IC5.QB, RN2B.2; no longer R17.1, T3.B
- net N$14: now also IC5.QA, RN2A.2; no longer K22.S, X7-1.S
- net N$15: now also JP3.1, RN2B.1, T2.G; no longer K32.S, X9-1.S
- net N$16: now also DF1.A, S12.1, T1.M2, V1.2; no longer K12.S, X8-1.S
- net N$17: now also DF2.A, S12.2, T2.M2, V2.2; no longer R25.1, T2.B
- net N$18: now also DF3.A, S34.1, T3.M2, V3.2; no longer R9.1, SELECT.3, SELECT.4
- net N$19: now also JP4.1, RN2C.1, T3.G; no longer K12.P, K12.P@1, X8-3.S
- net N$2: now also C2.+, F1.1, IC1.FB, L1'.2, L1.2; no longer D1.A, K21.2, R15.2, T1.C
- net N$20: now also DF4.A, S34.2, T4.M2, V4.2; no longer K12.O, X8-2.S
- net N$21: now also JP5.1, RN2D.1, T4.G; no longer LED1.C, R18.1
- net N$22: now also DF5.A, S56.1, T5.M2, V5.2; no longer R2.1, U$2.CLK
- net N$23: now also DF6.A, S56.2, T6.M2, V6.2; no longer R5.1, U$2.CE
- net N$24: now also DF7.A, S78.1, T7.M2, V7.2; no longer R4.1, U$2.DC
- net N$25: now also DF8.A, S78.2, T8.M2, V8.2; no longer R3.1, U$2.DIN
- net N$26: now also JP6.1, RN3A.1, T5.G; no longer T4.C, U$2.BL
- net N$27: now also JP7.1, RN3B.1, T6.G; no longer LED1.A
- net N$28: now also JP8.1, RN3C.1, T7.G; no longer K32.P, K32.P@1, X9-3.S
- net N$29: now also JP9.1, RN3D.1, T8.G; no longer K32.O, X9-2.S
- net N$3: now also JP2.1, RN2A.1, T1.G; no longer R14.1, T1.B
- net N$30: now also X1'1.2, X1.1; no longer X2.1
- net N$38: now also R-.2; no longer R8.2
- net N$4: now also IC5.QF, RN3B.2; no longer K22.P, K22.P@1, X7-3.S
- net N$41: now also CX1.1, X2'.2, X2.2; no longer C1.1, X1.2
- net N$42: now also CX2.1, X2'.1, X2.1; no longer C2.1, X1.1
- net N$45: now also R+.2; no longer R7.2
- net N$5: now also IC5.QG, RN3C.2; no longer K22.O, X7-2.S
- net N$54: now also RN4C.2, RN4D.2; no longer R19.2, R20.1
- net N$6: now also J0.2, J2.P; no longer DOWN.3, DOWN.4, R10.2, R11.1
- net N$7: now also IC5.QH, RN3D.2; no longer LED2.C, R15.1
- net N$8: now also X1'1.1, X1.2; no longer X2.2
- net N$9: now also D3.C, IC1.OUT, L1'.1, L1.1; no longer R11.2, R12.1, UP.3, UP.4
- net RD+: now also RN4D.1; no longer R20.2
- net RD-: now also RN4C.1; no longer R19.1
- net RESET: now also IC8.RESET, RN1A.1
- net SCK: now also IC6.SCK, IC8.(PCINT15/SCK)PB7, U1.SCK
- net SCL: now also IC8.(PCINT16/SCL)PC0, P0.10, RN1C.1; no longer R24.1, U1.PC5(ADC5/SCL)
- net SDA: now also IC8.(PCINT17/SDA)PC1, P0.11, RN1D.1; no longer R23.1, U1.PC4(ADC4/SDA)
- net TCT: now also RN4A.2, RN4B.2; no longer R21.2, R22.1
- net TD+: now also RN4A.1; no longer R22.2
- net TD-: now also RN4B.1; no longer R21.1
- net VCC: now also C3.+, C4.1, C9.1, EXTOUT.1, IC2.OUT@1, IC5.SCL, IC5.VCC, IC6.VDD, IC6.VDDOSC, IC6.VDDPLL, IC6.VDDRX, IC6.VDDTX, IC7.VCC, IC8.AVCC, IC8.VCC, IC8.VCC@1, IC8.VCC@2, P0.12, P1.1, RN1A.2, RN1B.2, RPR.2, U1.VCC; no longer R13.2, R16.2, U1.AVCC, U1.VCC@1, U1.VCC@2
- net VIN: now also C6.1, D2.C, F1.2, IC2.IN, IC3.VCC, LCD.A, LCD.VDD, P0.13, P4.2, P5.1, RN1C.2, RN1D.2
Other:
- note added: "!OE"
- note added: "3.3V"
- note added: "330x4 Isolated ResNet"
- note added: "5V"
- note added: "Clock"
- note added: "DB4"
- note added: "DB5"
- note added: "DB6"
- note added: "DB7"
- note added: "Data"
- note added: "EN_ETHER"
- note added: "Ext. Board Portion"
- note added: "LCD Display"
- note added: "LCD_BKLIGHT"
- note added: "LCD_E"
- note added: "LCD_RS"
- note added: "LCD_VO"
- note added: "Latch"
- note added: "PR"
- note added: "Power Supply"
- note added: "RAINSENSE"
- note added: "RF"
- note added: "SD_SEL"
- note added: "Valve Driver"
- moved on the sheet: C3, C4, C5, C6, C9, D1, D2, D3, IC2, RBS, RUSB
