File: v.2/kolektorius_v2.brd (EAGLE design)
At the start: 100 x 50 mm, 44 parts, among them IC2 LM1117-33, IC3 DS1307, IC6 ENC28J60, IC7 ATTINY45SO8S2, K1 JRC-21F_4100, K2 JRC-21F_4100, U1 ATMEGA328P, X1 25MHz, X2 32.768kHz

Commit message: judam pirmyn
Parts:
- removed COM, J1: (no value), SparkFun:SCREWTERMINAL-5MM-2
- removed RN3: 49.9, resistor-dil:EXB38V
- removed RN4: (no value), resistor-dil:EXB38V
- removed S1, S2, S3, S4, S5: (no value), SparkFun-Electromechanical:TACTILE-PTH
- added CX3, CX4: 18p, resistor:C0805
- added CX5, CX6: 100n, resistor:C0805
- added D1, D2: (no value), adafruit:DO-1N4148
- added DOWN, LEFT, RESET, RIGHT, SELECT, UP: (no value), SparkFun-Electromechanical:TACTILE-PTH
- added JP1, JP3: M022.54MM_SCREWTERM, SparkFun-Connectors:1X02_2.54_SCREWTERM
- added LED1, LED2: (no value), adafruit:1206
- added R10: 1k, rcl:R0805
- added R11: 620, rcl:R0805
- added R12: 330, rcl:R0805
- added R13: 2k, rcl:R0805
- added R14, R17, R9: 3k3, rcl:R0805
- added R15, R18: 470, rcl:R0805
- added R16, R23, R24: 10k, rcl:R0805
- added R19, R20, R21, R22: 49, rcl:R0805
- added T1, T3: 2N2222, adafruit:TO92-EBC-OVAL
- added X3: 25MHz, SparkFun:HC49US
- added X4, X5, X6: (no value), con-phoenix-254:3POL254
- K1, K2: value JRC-21F_4100 -> G5V1; device relay1:JRC-21F_4100 -> relay:G5V1
- moved CX2 94.4 mm to (20.9, 8.94)
- moved CX1 88.7 mm to (20.7, 11.5)
- moved X1 80.9 mm to (12.1, 10.7), turned to 0 degrees
- moved BAT1 59.5 mm to (33.9, 27.6)
- moved IC2 50.4 mm to (3.60, 13.4)
- moved L2 45.2 mm to (55.2, 26.4), turned to 270 degrees
- moved REB 42.2 mm to (44.4, 20.1)
- moved SJ1 40.5 mm to (22.8, 21.2)
- moved RBS 37.8 mm to (44.6, 23.1), turned to 180 degrees
- moved IC7 33.3 mm to (30.8, 14.7)
- moved C9 22.7 mm to (2.08, 45.9)
- moved RUSB 22.6 mm to (15.7, 1.17)
- moved K2 19.9 mm to (77.5, 12.7), turned to 270 degrees
- moved R7 12.8 mm to (64.8, 27.9)
- moved R8 12.0 mm to (57.1, 26.7)
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Connections:
- net N$10 renamed A4
- net N$11 renamed A5
- net N$13 renamed A7
- net N$3 renamed A0
- net N$4 renamed A1
- net N$5 renamed A2
- net N$7 renamed A3
- removed net 24VAC: COM.1, COM.2
- removed net INT1: J1.2
- removed net N$28: U1.5
- removed net N$29: U1.3
- removed net N$31: U1.21
- removed net N$40: U1.6
- removed net N$43: U1.4
- removed net N$44: U1.18
- new net A6: R12.2, R13.1, RIGHT.3, RIGHT.4, U1.19
- new net DTR: CX5.1
- new net N$1: LEFT.3, LEFT.4, R10.1, R9.2
- new net N$10: R14.2
- new net N$13: R17.1, T3.B
- new net N$18: R9.1, SELECT.3, SELECT.4
- new net N$19: JP3.P2, K1.5, K1.6
- new net N$2: D1.A, K2.9, R15.2, T1.C
- new net N$20: JP3.P1, K1.1
- new net N$21: LED1.C, R18.1
- new net N$27: R17.2
- new net N$3: R14.1, T1.B
- new net N$4: JP1.P2, K2.5, K2.6
- new net N$5: JP1.P1, K2.1
- new net N$6: DOWN.3, DOWN.4, R10.2, R11.1
- new net N$7: LED2.C, R15.1
- new net N$9: R11.2, R12.1, UP.3, UP.4
- net GND: now also CX3.1, CX4.1, CX6.2, DOWN.1, DOWN.2, LEFT.1, LEFT.2, RESET.1, RESET.2, RIGHT.1, SELECT.1, SELECT.2, T1.E, T3.E, U1.21, U1.3, U1.5, UP.1, UP.2; no longer J1.1
- net N$12: now also D2.A, K1.9, R18.2, T3.C; no longer U1.19
- net N$32: now also CX4.2, X3.1
- net N$33: now also CX3.2, X3.2
- net N$35: now also CX6.1
- net N$46: now also CX5.2, R16.1, RESET.3, RESET.4
- net N$54: now also R19.2, R20.1; no longer RN3.5, RN3.6
- net RD+: now also R20.2; no longer RN3.4
- net RD-: now also R19.1; no longer RN3.3
- net SCL: now also R24.1; no longer RN4.1
- net SDA: now also R23.1; no longer RN4.2
- net TCT: now also R21.2, R22.1; no longer RN3.7, RN3.8
- net TD+: now also R22.2; no longer RN3.2
- net TD-: now also R21.1; no longer RN3.1
- net VCC: now also C9.1, D1.C, D2.C, IC3.8, K1.2, K2.2, LED1.A, LED2.A, R13.2, R16.2, R23.2, R24.2, U1.18, U1.4, U1.6
- net VIN: no longer C9.1, IC3.8, RN4.7, RN4.8
Routing:
- net GND: track 17.6 -> 349.3 mm, vias 0 -> 5
- net VCC: track 0.00 -> 264.0 mm, vias 0 -> 2
- net N$46: track 0.00 -> 92.1 mm, vias 0 -> 1
- net A6: track 0.00 -> 84.3 mm, vias 0 -> 1
- net N$45: track 0.00 -> 83.5 mm, vias 0 -> 2
- net TD+: track 0.00 -> 74.1 mm, vias 0 -> 3
- net TD-: track 0.00 -> 71.0 mm, vias 0 -> 1
- net LEDA: track 0.00 -> 69.1 mm, vias 0 -> 2
- net TCT: track 0.00 -> 62.9 mm, vias 0 -> 1
- net RD-: track 0.00 -> 58.7 mm, vias 0 -> 2
- net RD+: track 0.00 -> 57.1 mm, vias 0 -> 3
- net N$52: track 0.00 -> 50.0 mm, vias 0 -> 1
- net D-: track 0.00 -> 41.8 mm, vias 0 -> 2
- net D+: track 0.00 -> 40.1 mm, vias 0 -> 2
- net N$59: track 0.00 -> 37.9 mm, vias 0 -> 2
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
Commit message: ...
Parts:
- removed IC3: DS1307, adafruit:SO08
- removed IC7: ATTINY45SO8S2, SparkFun:SO8S2
- added ATTINY: ATTINY45SO8S2, SparkFun:SO8S2
- added DS1307: DS1307, adafruit:SO08
- moved C9 43.5 mm to (38.0, 21.4)
- moved R23 38.6 mm to (37.9, 21.8)
- moved R24 38.4 mm to (33.4, 19.9)
- moved X2 37.8 mm to (40.3, 25.2), turned to 270 degrees
- moved CX4 20.8 mm to (-9.36, 36.8)
- moved C8 19.9 mm to (-11.8, 29.4)
- moved R22 19.8 mm to (9.97, 12.3), turned to 90 degrees
- moved R21 19.7 mm to (8.10, 12.3), turned to 270 degrees
- moved R20 17.6 mm to (-10.0, 26.7)
- moved R19 17.1 mm to (-6.85, 27.9)
- moved IC6 16.4 mm to (6.28, 34.1), turned to 90 degrees
- moved CAP 11.7 mm to (0.92, 21.2)
- moved BAT1 9.02 mm to (35.8, 36.4)
- moved X3 7.62 mm to (23.6, 30.7), turned to 270 degrees
- moved U1 6.91 mm to (15.3, 24.4), turned to 180 degrees
Connections:
- removed net A4: U1.27
- removed net A5: U1.28
- net D+: now also ATTINY.2; no longer IC7.2
- net D-: now also ATTINY.3; no longer IC7.3
- net GND: now also ATTINY.4, DS1307.4; no longer IC3.4, IC7.4
- net MISO: now also ATTINY.6; no longer IC7.6
- net MOSI: now also ATTINY.5; no longer IC7.5
- net N$30: now also DS1307.2; no longer IC3.2
- net N$36: now also DS1307.3; no longer IC3.3
- net N$52: now also ATTINY.1; no longer IC7.1
- net N$8: now also DS1307.1; no longer IC3.1
- net SCK: now also ATTINY.7; no longer IC7.7
- net SCL: now also DS1307.6, U1.28; no longer IC3.6
- net SDA: now also DS1307.5, U1.27; no longer IC3.5
- net VCC: now also ATTINY.8, DS1307.8; no longer IC3.8, IC7.8
Routing:
- net GND: track 349.3 -> 0.00 mm, vias 5 -> 0
- net VCC: track 264.0 -> 0.00 mm, vias 2 -> 0
- net N$46: track 92.1 -> 0.00 mm, vias 1 -> 0
- net A6: track 84.3 -> 0.00 mm, vias 1 -> 0
- net N$45: track 83.5 -> 0.00 mm, vias 2 -> 0
- net TD+: track 74.1 -> 0.00 mm, vias 3 -> 0
- net TD-: track 71.0 -> 0.00 mm, vias 1 -> 0
- net LEDA: track 69.1 -> 0.00 mm, vias 2 -> 0
- net TCT: track 62.9 -> 0.00 mm, vias 1 -> 0
- net RD-: track 58.7 -> 0.00 mm, vias 2 -> 0
- net RD+: track 57.1 -> 0.00 mm, vias 3 -> 0
- net N$52: track 50.0 -> 0.00 mm, vias 1 -> 0
- net D-: track 41.8 -> 0.00 mm, vias 2 -> 0
- net D+: track 40.1 -> 0.00 mm, vias 2 -> 0
- net N$59: track 37.9 -> 0.00 mm, vias 2 -> 0
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
Commit message: pcb...
Parts:
- CX3, CX4: value 18p -> 22p
- moved R19 59.1 mm to (52.2, 30.0), flipped to the bottom, turned to 270 degrees
- moved R20 58.1 mm to (48.1, 26.4), flipped to the bottom, turned to 180 degrees
- moved R22 54.8 mm to (61.6, 30.6), flipped to the bottom
- moved R21 53.0 mm to (57.9, 30.6), flipped to the bottom
- moved CX6 49.2 mm to (1.91, 31.2), flipped to the bottom, turned to 270 degrees
- moved IC2 42.9 mm to (35.5, 42.1), turned to 0 degrees
- moved X2 38.2 mm to (2.51, 19.5)
- moved X1 37.4 mm to (43.5, 31.0), turned to 90 degrees
- moved CX2 35.5 mm to (47.1, 32.9), flipped to the bottom, turned to 90 degrees
- moved REA 35.2 mm to (43.3, 40.1), flipped to the bottom, turned to 180 degrees
- moved CX1 34.8 mm to (43.4, 37.9), flipped to the bottom
- moved CX4 31.8 mm to (22.1, 32.4), flipped to the bottom
- moved CAP 31.7 mm to (29.2, 35.6), flipped to the bottom, turned to 270 degrees
- moved IC6 29.7 mm to (35.9, 32.1), turned to 270 degrees
- moved DS1307 24.9 mm to (10.6, 18.4), turned to 180 degrees
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Routing:
- net GND: track 0.00 -> 334.8 mm, vias 0 -> 7
- net VCC: track 0.00 -> 232.3 mm, vias 0 -> 9
- net A6: track 0.00 -> 121.8 mm
- net N$46: track 0.00 -> 105.6 mm, vias 0 -> 1
- net N$45: track 0.00 -> 82.9 mm, vias 0 -> 2
- net TCT: track 0.00 -> 62.6 mm, vias 0 -> 2
- net N$54: track 0.00 -> 50.6 mm
- net SCL: track 0.00 -> 47.7 mm, vias 0 -> 1
- net LEDB: track 0.00 -> 40.4 mm, vias 0 -> 1
- net SDA: track 0.00 -> 37.2 mm, vias 0 -> 1
- net VIN: track 0.00 -> 35.1 mm, vias 0 -> 1
- net D11: track 0.00 -> 34.6 mm
- net RD+: track 0.00 -> 34.6 mm, vias 0 -> 3
- net D-: track 0.00 -> 32.2 mm, vias 0 -> 1
- net N$9: track 0.00 -> 31.0 mm, vias 0 -> 2
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
Commit message: pcb..
Parts:
- moved REB 27.3 mm to (45.0, 47.4), turned to 180 degrees
- moved REA 15.7 mm to (57.9, 45.8)
- moved RBS 2.05 mm to (44.2, 20.4), turned to 0 degrees
- moved X2 1.80 mm to (2.69, 17.8), turned to 0 degrees
- moved C7 1.48 mm to (5.36, 25.5), turned to 90 degrees
- moved R16 1.42 mm to (95.9, 2.54), turned to 180 degrees
- moved C8 0.40 mm to (8.21, 24.4), turned to 180 degrees
- flipped LED1 to the top
- flipped LED2 to the top
Routing:
- net RD+: track 34.6 -> 140.5 mm, vias 3 -> 5
- net VCC: track 232.3 -> 271.9 mm, vias 9 -> 13
- net LEDB: track 40.4 -> 2.98 mm, vias 1 -> 0
- net GND: track 334.8 -> 359.4 mm, vias 7 -> 9
- net N$54: track 50.6 -> 73.8 mm, vias 0 -> 4
- net LEDA: track 23.2 -> 3.95 mm
- net N$34: track 6.21 -> 22.9 mm
- net TCT: track 62.6 -> 75.1 mm, vias 2 -> 5
- net N$8: track 12.5 -> 20.5 mm
- net N$42: track 14.1 -> 20.2 mm, vias 2 -> 3
- net N$37: track 20.5 -> 15.2 mm
- net N$36: track 8.17 -> 12.7 mm
- net N$59: track 21.2 -> 16.9 mm, vias 3 -> 1
- net N$30: track 10.8 -> 14.7 mm
- net N$46: track 105.6 -> 108.7 mm, vias 1 -> 2
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
Commit message: pcb
Routing:
- net N$32: track 13.3 -> 8.89 mm, vias 0 -> 2
- net N$7: track 5.55 -> 2.86 mm
- net N$21: track 5.55 -> 2.86 mm
- net N$46: track 108.7 -> 108.0 mm
- net D8: vias 2 -> 3

Commit message: pcb
Parts:
- removed JP1, JP3: M022.54MM_SCREWTERM, SparkFun-Connectors:1X02_2.54_SCREWTERM
- added D3: (no value), adafruit:DO-1N4148
- added K3: G5V1, relay:G5V1
- added LED3: (no value), adafruit:1206
- added R25, R28: 3k3, rcl:R0805
- added R26: 470, rcl:R0805
- added T2, T4: 2N2222, adafruit:TO92-EBC-OVAL
- added X7, X8, X9: 22-23-2031, con-molex:22-23-2031
- moved RESET 41.3 mm to (92.1, 42.9), turned to 0 degrees
- moved R16 33.7 mm to (96.5, 36.2), turned to 270 degrees
- moved X5 26.2 mm to (34.7, 1.12)
- moved CX5 21.4 mm to (75.2, 21.4)
- moved X6 15.4 mm to (53.2, 1.12), flipped to the bottom
- moved R14 11.5 mm to (80.0, 20.3)
- moved X4 9.35 mm to (44.0, 1.12)
- moved R17 7.63 mm to (98.1, 23.7), turned to 90 degrees
- moved R1 2.84 mm to (27.9, 39.4), turned to 90 degrees
- moved IC2 1.27 mm to (36.7, 42.1)
Connections:
- removed net N$10: R14.2
- removed net N$27: R17.2
- removed net N$51: R1.2
- new net D0: R25.2, U1.30
- new net D1: U1.31, X4.2
- new net D2: U1.32, X6.2
- new net N$11: D3.A, K3.9, R26.2, T2.C
- new net N$17: R25.1, T2.B
- new net N$28: K3.5, K3.6, X9.3
- new net N$29: K3.1, X9.2
- new net N$31: LED3.C, R26.1
- new net N$44: R1.2, T4.B
- net A1: now also X5.2
- net A2: now also R17.2
- net A3: now also R14.2
- net D10: now also R1.1, R28.2
- net GND: now also T2.E, T4.E, X4.1, X5.1, X6.1
- net N$14: now also K2.10, X7.1; no longer U1.30
- net N$15: now also K3.10, X9.1; no longer U1.31
- net N$16: now also K1.10, X8.1; no longer U1.32
- net N$19: now also X8.3; no longer JP3.P2
- net N$20: now also X8.2; no longer JP3.P1
- net N$26: now also T4.C; no longer R1.1
- net N$4: now also X7.3; no longer JP1.P2
- net N$5: now also X7.2; no longer JP1.P1
- net VCC: now also D3.C, K3.2, LED3.A, R28.1, X4.3, X5.3, X6.3
Routing:
- net A2: track 0.00 -> 120.5 mm, vias 0 -> 2
- net RD+: track 140.5 -> 33.8 mm, vias 5 -> 3
- net A3: track 0.00 -> 94.1 mm, vias 0 -> 3
- net D0: track 0.00 -> 71.2 mm, vias 0 -> 3
- net D2: track 0.00 -> 53.4 mm, vias 0 -> 5
- net VCC: track 271.9 -> 325.1 mm, vias 13 -> 7
- net A1: track 0.00 -> 47.1 mm, vias 0 -> 4
- net D1: track 0.00 -> 44.7 mm, vias 0 -> 3
- net D10: track 0.00 -> 26.0 mm, vias 0 -> 2
- net N$54: track 73.8 -> 50.4 mm
- net A6: track 121.8 -> 102.0 mm, vias 0 -> 1
- net N$29: track 0.00 -> 16.3 mm
- net N$15: track 0.00 -> 16.2 mm
- net N$14: track 0.00 -> 16.2 mm
- net N$16: track 0.00 -> 16.2 mm
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
Commit message: pcb
Parts:
- moved X4 1.27 mm to (44.0, 2.39)
- moved X5 1.27 mm to (34.7, 2.39)
- moved X6 1.27 mm to (53.2, 2.39)
- moved C3 0.11 mm to (6.42, 3.85), turned to 0 degrees
Routing:
- net VCC: track 325.1 -> 293.4 mm, vias 7 -> 9
- net GND: track 358.1 -> 340.5 mm, vias 6 -> 5
- net A6: track 102.0 -> 117.3 mm
- net A3: track 94.1 -> 80.0 mm
- net D0: track 71.2 -> 58.7 mm
- net A2: track 120.5 -> 111.3 mm, vias 2 -> 4
- net D8: track 34.8 -> 25.7 mm, vias 0 -> 2
- net D13: track 29.1 -> 37.6 mm
- net D12: track 35.9 -> 31.0 mm, vias 0 -> 2
- net D-: track 35.1 -> 30.9 mm
- net N$46: track 110.0 -> 105.8 mm, vias 2 -> 4
- net N$33: track 11.3 -> 15.3 mm, vias 2 -> 0
- net RD-: track 24.5 -> 27.9 mm
- net RD+: track 33.8 -> 31.6 mm
- net N$38: track 24.2 -> 22.3 mm, vias 1 -> 0
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