File: v.2/kolektorius_v2.brd (EAGLE design)
At the start: 100 x 50 mm, 81 parts, among them IC2 LM1117-33, IC6 ENC28J60, K1 G5V1, K2 G5V1, K3 G5V1, T1 2N2222, T2 2N2222, T3 2N2222, T4 2N2222, U1 ATMEGA328P, X1 25MHz, X2 32.768kHz, X3 25MHz, X7 22-23-2031, X8 22-23-2031, X9 22-23-2031

Commit message: pcb
prie pabaigos...
Parts:
- removed CX1, CX2: 18p, resistor:C0805
- removed CX3, CX4: 22p, resistor:C0805
- removed DS1307: DS1307, adafruit:SO08
- removed IC6: ENC28J60, SparkFun-DigitalIC:SSOP28DB
- removed L2: Bead, rcl:R0805
- removed R28: 3k3, rcl:R0805
- added C1: 100u, resistor:E2-5
- added C4, C5: 0.1µ, resistor:C0805
- added C6: 18p, resistor:C0805
- added DS1: DS1307, adafruit:SO08
- added IC1: LM1117-33, SparkFun:SOT223
- added L1: Bead, rcl:R0805
- added X10: 22-23-2031, con-molex:22-23-2031
- added X11: (no value), con-phoenix-254:2POL254
- C3: value 100u -> 0.1u; device resistor:PANASONIC_D -> rcl:C0805
- C7: value 0.1µ -> 18p
- C8: value 0.1µ -> 22p
- C9: value 0.1u -> 22p; device rcl:C0805 -> resistor:C0805
- IC2: value LM1117-33 -> ENC28J60; device SparkFun:SOT223 -> SparkFun-DigitalIC:SSOP28DB
- R1, R3, R5: value 10k -> 470
- R10: value 1k -> 330
- R11: value 620 -> 3k3
- R12: value 330 -> 620
- R13: value 2k -> 1k
- R14: value 3k3 -> 49
- R15: value 470 -> 49
- R16: value 10k -> 49
- R17, R25: value 3k3 -> 10k
- R18: value 470 -> 47
- R19: value 49 -> 47
- R2, R4, R6: value 10k -> 3k3
- R21: value 49 -> 1k
- R22: value 49 -> 10k
- R26: value 470 -> 10k
- R7, R8: value 47 -> 10k
- R9: value 3k3 -> 2k
- X1: value 25MHz -> 32.768kHz; device SparkFun:HC49US -> crystal:TC26H
- X2: value 32.768kHz -> 25MHz; device crystal:TC26H -> SparkFun:HC49US
- X4: device con-phoenix-254:3POL254 -> con-phoenix-254:2POL254
- X7: value 22-23-2031 -> (none); device con-molex:22-23-2031 -> con-phoenix-254:3POL254
- moved T4 73.1 mm to (97.8, 17.8), turned to 270 degrees
- moved R1 72.5 mm to (95.2, 12.7)
- moved R2 71.6 mm to (92.5, 20.6), turned to 0 degrees
- moved R3 67.6 mm to (82.5, 12.7), turned to 90 degrees
- moved R4 64.5 mm to (80.0, 20.9), turned to 0 degrees
- moved R26 63.1 mm to (14.0, 41.9), turned to 270 degrees
- moved T1 61.4 mm to (29.2, 43.2), turned to 180 degrees
- moved R5 60.8 mm to (69.8, 12.7), turned to 90 degrees
- moved R6 57.1 mm to (67.3, 21.6), turned to 0 degrees
- moved USB 55.7 mm to (53.7, -1.93), turned to 0 degrees
- moved R25 55.2 mm to (16.5, 41.9), turned to 270 degrees
- moved R18 46.8 mm to (48.9, 6.35), turned to 180 degrees
- moved R16 44.0 mm to (52.9, 30.9)
- moved RUSB 42.7 mm to (48.9, 8.25), turned to 0 degrees
- moved R22 39.9 mm to (24.1, 41.9), turned to 270 degrees
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- renumbered CX6 to C2, RJ45 to RJ1, U$2 to U$1
Connections:
- removed net N$15 (its old number): K3.10, X9.1
- removed net N$28 (its old number): K3.5, K3.6, X9.3
- removed net N$29 (its old number): K3.1, X9.2
- new net +3V3: C1.+, IC1.4, IC2.15, IC2.19, IC2.20, IC2.25, IC2.28
- new net +5V: ATTINY.8, C3.1, D1.C, D2.C, D3.C, DS1.8, IC1.3, K1.2, K2.2, K3.2, L1.2, LED1.A, LED2.A, R7.2, R8.2, U$1.P$6, X11.2, X5.3, X6.3, X7.3
- new net N$16: K3.10, X10.1
- new net N$19: K3.5, K3.6, X10.3
- new net N$20: K3.1, X10.2
- new net N$27: LED3.A
- net A1: now also X6.2; no longer X5.2
- net A2: now also R2.2; no longer R17.2
- net A3: now also R4.2; no longer R14.2
- net A6: now also R10.2, R9.1; no longer R12.2, R13.1
- net D+: now also R19.1; no longer R8.1
- net D-: now also R18.1; no longer R7.1
- net D0: now also R6.2; no longer R25.2
- net D1: now also X5.2; no longer X4.2
- net D10: now also R21.2; no longer R1.1, R28.2
- net D11: now also IC2.7; no longer IC6.7
- net D12: now also IC2.6; no longer IC6.6
- net D13: now also IC2.8; no longer IC6.8
- net D2: now also X7.2; no longer X6.2
- net D3: now also R22.2; no longer R2.2
- net D4: now also R23.2; no longer R3.2
- net D5: now also R24.2; no longer R4.2
- net D6: now also R25.2; no longer R5.2
- net D7: now also R26.2; no longer R6.2
- net D8: now also IC2.9; no longer IC6.9
- net GND: now also C1.-, C3.2, C4.1, C5.1, C6.2, C7.2, C9.1, DS1.4, IC1.1, IC2.11, IC2.18, IC2.2, IC2.21, IC2.22, X11.1, X7.1; no longer C3.-, C7.1, C9.2, CX1.2, CX2.2, CX3.1, CX4.1, DS1307.4, IC2.1, IC6.11, IC6.18, IC6.2, IC6.21, IC6.22, X4.1
- net N$1: now also R11.2, R13.1; no longer R10.1, R9.2
- net N$11: now also D1.A, K1.9, R5.2; no longer D3.A, K3.9, R26.2
- net N$12: now also D3.A, K3.9, R1.2, T4.C; no longer D2.A, K1.9, R18.2, T3.C
- net N$13: now also R2.1, T4.B; no longer R17.1, T3.B
- net N$14: now also X9.1; no longer X7.1
- net N$17: now also R6.1; no longer R25.1
- net N$18: now also R11.1; no longer R9.1
- net N$2: now also D2.A, R3.2, T3.C; no longer D1.A, R15.2, T1.C
- net N$21: now also LED3.C, R1.1; no longer LED1.C, R18.1
- net N$22: now also R22.1; no longer R2.1
- net N$23: now also R25.1; no longer R5.1
- net N$24: now also R24.1; no longer R4.1
- net N$25: now also R23.1; no longer R3.1
- net N$26: now also T1.C; no longer T4.C
- net N$3: now also R4.1, T3.B; no longer R14.1, T1.B
- net N$30: now also DS1.2, X1.1; no longer DS1307.2, X2.1
- net N$31: now also LED1.C, R5.1; no longer LED3.C, R26.1
- net N$32: now also C9.2, X2.1; no longer CX4.2, X3.1
- net N$33: now also C8.2, X2.2; no longer CX3.2, X3.2
- net N$34: now also IC2.27; no longer IC6.27
- net N$36: now also DS1.3; no longer DS1307.3
- net N$37: now also IC2.26; no longer IC6.26
- net N$38: now also R19.2; no longer R8.2
- net N$39: now also IC2.1; no longer IC6.1
- net N$4: now also X9.3; no longer X7.3
- net N$41: now also C6.1, IC2.24, X3.2; no longer CX1.1, IC6.24, X1.2
- net N$42: now also C7.1, IC2.23, X3.1; no longer CX2.1, IC6.23, X1.1
- net N$44: now also R21.1, T1.B; no longer R1.2, T4.B
- net N$45: now also R18.2; no longer R7.2
- net N$46: now also R17.1; no longer R16.1
- net N$5: now also X9.2; no longer X7.2
- net N$54: now also C5.2, R15.1, R16.2; no longer C7.2, R19.2, R20.1
- net N$59: now also IC2.14; no longer IC6.14
- net N$6: now also R12.1, R13.2; no longer R10.2, R11.1
- net N$7: now also R3.1; no longer R15.1
- net N$8: now also DS1.1, X1.2; no longer DS1307.1, X2.2
- net N$9: now also R10.1, R12.2; no longer R11.2, R12.1
- net RD+: now also IC2.13, R15.2; no longer IC6.13, R20.2
- net RD-: now also IC2.12, R16.1; no longer IC6.12, R19.1
- net RESET: now also IC2.10; no longer IC6.10
- net SCL: now also DS1.6, R7.1; no longer DS1307.6, R24.1
- net SDA: now also DS1.5, R8.1; no longer DS1307.5, R23.1
- net TCT: now also C4.2, L1.1, R14.2, R20.1; no longer C8.2, L2.1, R21.2, R22.1
- net TD+: now also IC2.17, R20.2; no longer IC6.17, R22.2
- net TD-: now also IC2.16, R14.1; no longer IC6.16, R21.1
- net V$: now also R26.1; no longer R6.1
- net VCC: now also R17.2, R9.2; no longer ATTINY.8, C3.+, C9.1, D1.C, D2.C, D3.C, DS1307.8, IC2.4, IC6.15, IC6.19, IC6.20, IC6.25, IC6.28, K1.2, K2.2, K3.2, L2.2, LED1.A, LED2.A, LED3.A, R13.2, R16.2, R23.2, R24.2, R28.1, U$1.P$6, X4.3, X5.3, X6.3
Routing:
- net GND: track 351.9 -> 77.3 mm, vias 5 -> 4
- net +5V: track 0.00 -> 216.4 mm, vias 0 -> 1
- net VCC: track 310.0 -> 128.7 mm, vias 8 -> 4
- net D+: track 40.1 -> 5.55 mm
- net D-: track 46.6 -> 12.2 mm, vias 3 -> 1
- net +3V3: track 0.00 -> 30.3 mm
- net VIN: track 35.7 -> 12.5 mm, vias 1 -> 0
- net N$20: track 0.00 -> 16.3 mm
- net N$29 (its old number): track 16.3 -> 0.00 mm
- net N$15 (its old number): track 16.2 -> 0.00 mm
- net N$16: track 0.00 -> 16.2 mm
- net D1: track 42.9 -> 31.1 mm, vias 1 -> 0
- net D2: track 52.6 -> 41.1 mm, vias 0 -> 1
- net D11: track 30.1 -> 41.0 mm, vias 2 -> 0
- net N$38: track 3.64 -> 14.4 mm
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- added copper zone on layer 1, net +3V3
- added copper zone on layer 16, net GND

Commit message: pcb
Parts:
- added C10, C11, C12, C14, C15, C16: 100n, resistor:C0805
Connections:
- net +3V3: now also C14.1
- net +5V: now also C11.2, C12.2, C15.1, C16.1
- net GND: now also C10.2, C11.1, C12.1, C14.2, C15.2, C16.2
- net VCC: now also C10.1
Routing:
- net GND: track 77.3 -> 409.1 mm, vias 4 -> 8
- net +5V: track 216.4 -> 267.5 mm
- net VCC: track 128.7 -> 136.9 mm
- net +3V3: track 30.3 -> 33.4 mm, vias 0 -> 1
- removed copper zone on layer 16, net GND
Other:
- board size 100 x 50 mm -> 100 x 50.2 mm

Commit message: pcb prie pabaigos
Parts:
- X2: value 25MHz -> 16MHz
- moved C15 1.97 mm to (32.2, 9.40)
- moved R14 0.05 mm to (61.0, 33.2)
Routing:
- net GND: track 409.1 -> 407.1 mm
- net +5V: track 267.5 -> 266.8 mm
- net A1: vias 1 -> 2
Other:
- board text added: "2014.02"
- board text removed: "(2014.02)"

Commit message: xxx
Parts:
- moved R17 30.5 mm to (66.0, 35.6)
- moved RESET 21.7 mm to (70.5, 41.0)
Routing:
- net N$46: track 112.9 -> 76.4 mm, vias 1 -> 2
- net GND: track 407.1 -> 401.1 mm
- net A6: track 113.7 -> 118.2 mm
- net VCC: track 136.9 -> 138.2 mm

Commit message: pabaiga
Parts:
- moved X11 3.81 mm to (8.26, 1.91)
Routing:
- net +5V: track 266.8 -> 251.4 mm, vias 1 -> 2
- net GND: track 401.1 -> 403.4 mm, vias 8 -> 6
