File: v.2/kolektorius_v21.brd (EAGLE design)
At the start: 100 x 50.2 mm, 88 parts, among them IC1 LM1117-33, IC2 ENC28J60, K1 G5V1, K2 G5V1, K3 G5V1, T1 2N2222, T2 2N2222, T3 2N2222, T4 2N2222, U1 ATMEGA328P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

Commit message: pcb
Parts:
- moved C11 1.27 mm to (3.81, 26.0)
Routing:
- net +5V: track 265.2 -> 267.5 mm
- net GND: track 407.8 -> 409.1 mm
Changed lines of the file:
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@@
 <grid distance="0.635" unitdist="mm" unit="mm" style="lines" multiple="1" display="yes" altdistance="0.025" altunitdist="inch" altunit="mm"/>
 <layers>
-<layer number="1" name="Top" color="4" fill="1" visible="yes" active="yes"/>
+<layer number="1" name="Top" color="4" fill="1" visible="no" active="yes"/>
 <layer number="2" name="Route2" color="1" fill="3" visible="no" active="no"/>
 <layer number="3" name="Route3" color="4" fill="3" visible="no" active="no"/>
@@
 <layer number="19" name="Unrouted" color="6" fill="1" visible="yes" active="yes"/>
 <layer number="20" name="Dimension" color="15" fill="1" visible="yes" active="yes"/>
-<layer number="21" name="tPlace" color="7" fill="1" visible="yes" active="yes"/>
+<layer number="21" name="tPlace" color="7" fill="1" visible="no" active="yes"/>
 <layer number="22" name="bPlace" color="7" fill="1" visible="yes" active="yes"/>
-<layer number="23" name="tOrigins" color="15" fill="1" visible="yes" active="yes"/>
+<layer number="23" name="tOrigins" color="15" fill="1" visible="no" active="yes"/>
 <layer number="24" name="bOrigins" color="15" fill="1" visible="yes" active="yes"/>
-<layer number="25" name="tNames" color="7" fill="1" visible="yes" active="yes"/>
+<layer number="25" name="tNames" color="7" fill="1" visible="no" active="yes"/>
 <layer number="26" name="bNames" color="7" fill="1" visible="yes" active="yes"/>
-<layer number="27" name="tValues" color="7" fill="1" visible="yes" active="yes"/>
+<layer number="27" name="tValues" color="7" fill="1" visible="no" active="yes"/>
 <layer number="28" name="bValues" color="7" fill="1" visible="yes" active="yes"/>
 <layer number="29" name="tStop" color="7" fill="3" visible="no" active="yes"/>
@@
 <element name="R23" library="rcl" package="R0805" value="10k" x="21.59" y="41.91" smashed="yes" rot="MR270">
 <attribute name="NAME" x="21.59" y="40.005" size="1.27" layer="26" rot="MR270"/>
-<attribute name="VALUE" x="24.13" y="42.545" size="1.27" layer="28" rot="MR270"/>
+<attribute name="VALUE" x="20.955" y="44.45" size="1.27" layer="28" rot="MR270"/>
 </element>
 <element name="R24" library="rcl" package="R0805" value="10k" x="19.05" y="41.91" smashed="yes" rot="MR270">
 <attribute name="NAME" x="19.05" y="40.005" size="1.27" layer="26" rot="MR270"/>
-<attribute name="VALUE" x="21.59" y="42.545" size="1.27" layer="28" rot="MR270"/>
+<attribute name="VALUE" x="18.415" y="44.45" size="1.27" layer="28" rot="MR270"/>
 </element>
 <element name="R25" library="rcl" package="R0805" value="10k" x="16.51" y="41.91" smashed="yes" rot="MR270">
 <attribute name="NAME" x="16.51" y="40.005" size="1.27" layer="26" rot="MR270"/>
-<attribute name="VALUE" x="19.05" y="42.545" size="1.27" layer="28" rot="MR270"/>
+<attribute name="VALUE" x="15.875" y="44.45" size="1.27" layer="28" rot="MR270"/>
 </element>
 <element name="R22" library="rcl" package="R0805" value="10k" x="24.13" y="41.91" smashed="yes" rot="MR270">
 <attribute name="NAME" x="24.13" y="40.005" size="1.27" layer="26" rot="MR270"/>
-<attribute name="VALUE" x="26.67" y="42.545" size="1.27" layer="28" rot="MR270"/>
-</element>
-<element name="R26" library="rcl" package="R0805" value="10k" x="13.97" y="41.91" locked="yes" smashed="yes" rot="MR270">
+<attribute name="VALUE" x="23.495" y="44.45" size="1.27" layer="28" rot="MR270"/>
+</element>
+<element name="R26" library="rcl" package="R0805" value="10k" x="13.97" y="41.91" smashed="yes" rot="MR270">
 <attribute name="NAME" x="13.97" y="40.005" size="1.27" layer="26" rot="MR270"/>
-<attribute name="VALUE" x="16.51" y="42.545" size="1.27" layer="28" rot="MR270"/>
+<attribute name="VALUE" x="13.335" y="44.45" size="1.27" layer="28" rot="MR270"/>
 </element>
 <element name="R18" library="rcl" package="R0805" value="47" x="48.895" y="6.35" rot="MR180"/>
@@
 <element name="X2" library="SparkFun" package="HC49US" value="25MHz" x="18.56" y="31.98" rot="R270"/>
 <element name="C8" library="resistor" package="C0805" value="22p" x="20.92" y="29.79" smashed="yes" rot="MR270">
-<attribute name="NAME" x="24.349" y="30.679" size="1.27" layer="26" rot="MR270"/>
-<attribute name="VALUE" x="23.206" y="30.679" size="1.27" layer="28" rot="MR270"/>
+<attribute name="NAME" x="23.079" y="28.139" size="1.27" layer="26" rot="MR270"/>
+<attribute name="VALUE" x="23.206" y="31.949" size="1.27" layer="28" rot="MR270"/>
 </element>
 <element name="C9" library="resistor" package="C0805" value="22p" x="20.87" y="33.69" rot="MR90"/>
@@
 <element name="LED1" library="adafruit" package="1206" value="" x="69.85" y="7.62" rot="R90"/>
 <element name="T1" library="adafruit" package="TO92-EBC-OVAL" value="2N2222" x="29.21" y="43.18" smashed="yes" rot="R180">
-<attribute name="NAME" x="27.94" y="42.672" size="1.27" layer="25" ratio="10" rot="R180"/>
+<attribute name="NAME" x="31.75" y="43.942" size="1.27" layer="25" ratio="10" rot="R180"/>
 <attribute name="VALUE" x="31.75" y="47.752" size="1.27" layer="27" ratio="10" rot="R180"/>
 </element>
@@
 <element name="R21" library="rcl" package="R0805" value="1k" x="27.94" y="41.91" smashed="yes" rot="MR270">
 <attribute name="NAME" x="27.94" y="40.005" size="1.27" layer="26" rot="MR270"/>
-<attribute name="VALUE" x="30.48" y="42.545" size="1.27" layer="28" rot="MR270"/>
+<attribute name="VALUE" x="27.305" y="43.815" size="1.27" layer="28" rot="MR270"/>
 </element>
 <element name="C1" library="resistor" package="E2-5" value="100u" x="42.545" y="40.005" rot="R90"/>
@@
 <attribute name="OC_FARNELL" value="unknown" x="4.445" y="1.905" size="1.778" layer="27" display="off"/>
 </element>
-<element name="C10" library="resistor" package="C0805" value="100n" x="6.35" y="40.64" rot="MR0"/>
-<element name="C11" library="resistor" package="C0805" value="100n" x="2.54" y="26.035" rot="MR0"/>
+<element name="C10" library="resistor" package="C0805" value="100n" x="6.35" y="40.64" smashed="yes" rot="MR0">
+<attribute name="NAME" x="8.509" y="41.656" size="1.27" layer="26" rot="MR0"/>
+<attribute name="VALUE" x="4.699" y="41.529" size="1.27" layer="28" rot="MR0"/>
+</element>
+<element name="C11" library="resistor" package="C0805" value="100n" x="3.81" y="26.035" smashed="yes" rot="MR0">
+<attribute name="NAME" x="3.556" y="27.051" size="1.27" layer="26" rot="MR90"/>
+<attribute name="VALUE" x="2.921" y="31.369" size="1.27" layer="28" rot="MR270"/>
+</element>
 <element name="C12" library="resistor" package="C0805" value="100n" x="2.54" y="34.925" rot="MR90"/>
 <element name="C14" library="resistor" package="C0805" value="100n" x="36.195" y="29.21" rot="MR270"/>
 <element name="C15" library="resistor" package="C0805" value="100n" x="33.02" y="7.62" rot="MR270"/>
-<element name="C16" library="resistor" package="C0805" value="100n" x="6.985" y="8.89" rot="MR0"/>
+<element name="C16" library="resistor" package="C0805" value="100n" x="6.985" y="8.89" smashed="yes" rot="MR0">
+<attribute name="NAME" x="8.509" y="7.239" size="1.27" layer="26" rot="MR270"/>
+<attribute name="VALUE" x="4.826" y="12.319" size="1.27" layer="28" rot="MR270"/>
+</element>
 </elements>
 <signals>
@@
 <wire x1="9.1948" y1="30.9626" x2="9.3726" y2="30.861" width="0.4064" layer="16"/>
 <wire x1="3.4036" y1="34.0614" x2="3.4036" y2="26.035" width="0.4064" layer="16"/>
-<wire x1="3.4036" y1="26.035" x2="3.39" y2="26.035" width="0.4064" layer="16"/>
+<wire x1="3.4036" y1="26.035" x2="4.66" y2="26.035" width="0.4064" layer="16"/>
 <wire x1="5.5118" y1="34.0614" x2="5.5118" y2="40.64" width="0.4064" layer="16"/>
 <wire x1="5.5118" y1="40.64" x2="5.5" y2="40.64" width="0.4064" layer="16"/>
@@
 <wire x1="2.2352" y1="35.7632" x2="1.3716" y2="34.8996" width="0.4064" layer="16"/>
 <wire x1="2.54" y1="35.7632" x2="2.2352" y2="35.7632" width="0.4064" layer="16"/>
-<wire x1="1.6764" y1="26.035" x2="1.69" y2="26.035" width="0.4064" layer="16"/>
+<wire x1="1.6764" y1="26.035" x2="2.96" y2="26.035" width="0.4064" layer="16"/>
 <wire x1="2.54" y1="35.7632" x2="2.54" y2="35.775" width="0.4064" layer="16"/>
 <wire x1="1.778" y1="5.842" x2="1.778" y2="25.8572" width="0.4064" layer="16"/>
 <wire x1="5.715" y1="1.905" x2="3.4417" y2="4.1783" width="0.4064" layer="16"/>
 <wire x1="3.4417" y1="4.1783" x2="1.778" y2="5.842" width="0.4064" layer="16"/>
-<wire x1="1.778" y1="25.8572" x2="1.69" y2="26.035" width="0.4064" layer="16"/>
+<wire x1="1.778" y1="25.8572" x2="2.96" y2="26.035" width="0.4064" layer="16"/>
 <wire x1="56.8706" y1="20.5994" x2="56.8706" y2="20.7264" width="0.4064" layer="16"/>
 <wire x1="56.8706" y1="20.7264" x2="56.8706" y2="27.8892" width="0.4064" layer="16"/>
