File: v.2/kolektorius_v2-1.brd (EAGLE design)
At the start: 100 x 50 mm, 73 parts, among them IC2 LM1117-33, IC6 ENC28J60, K1 G5V1, K2 G5V1, T1 2N2222, T3 2N2222, U1 ATMEGA328P, X1 25MHz, X2 32.768kHz, X3 25MHz

Commit message: pcb
Parts:
- removed JP1, JP3: M022.54MM_SCREWTERM, SparkFun-Connectors:1X02_2.54_SCREWTERM
- added D3: (no value), adafruit:DO-1N4148
- added K3: G5V1, relay:G5V1
- added LED3: (no value), adafruit:1206
- added R25, R28: 3k3, rcl:R0805
- added R26: 470, rcl:R0805
- added T2, T4: 2N2222, adafruit:TO92-EBC-OVAL
- added X7, X8, X9: 22-23-2031, con-molex:22-23-2031
- moved RESET 41.3 mm to (92.1, 42.9), turned to 0 degrees
- moved R16 33.7 mm to (96.5, 36.2), turned to 270 degrees
- moved X5 26.3 mm to (34.7, 2.39)
- moved CX5 21.4 mm to (75.2, 21.4)
- moved X6 15.4 mm to (53.2, 2.39), flipped to the bottom
- moved X2 13.5 mm to (2.69, 17.8), turned to 0 degrees
- moved R14 11.5 mm to (80.0, 20.3)
- moved X4 9.41 mm to (44.0, 2.39)
- moved R17 7.63 mm to (98.1, 23.7), turned to 90 degrees
- moved R1 2.84 mm to (27.9, 39.4), turned to 90 degrees
- moved BAT1 2.43 mm to (20.0, 17.5)
- moved IC2 1.27 mm to (36.7, 42.1)
- moved C3 0.11 mm to (6.42, 3.85), turned to 0 degrees
Connections:
- removed net N$10: R14.2
- removed net N$27: R17.2
- removed net N$51: R1.2
- new net D0: R25.2, U1.30
- new net D1: U1.31, X4.2
- new net D2: U1.32, X6.2
- new net N$11: D3.A, K3.9, R26.2, T2.C
- new net N$17: R25.1, T2.B
- new net N$28: K3.5, K3.6, X9.3
- new net N$29: K3.1, X9.2
- new net N$31: LED3.C, R26.1
- new net N$44: R1.2, T4.B
- net A1: now also X5.2
- net A2: now also R17.2
- net A3: now also R14.2
- net D10: now also R1.1, R28.2
- net GND: now also T2.E, T4.E, X4.1, X5.1, X6.1
- net N$14: now also K2.10, X7.1; no longer U1.30
- net N$15: now also K3.10, X9.1; no longer U1.31
- net N$16: now also K1.10, X8.1; no longer U1.32
- net N$19: now also X8.3; no longer JP3.P2
- net N$20: now also X8.2; no longer JP3.P1
- net N$26: now also T4.C; no longer R1.1
- net N$4: now also X7.3; no longer JP1.P2
- net N$5: now also X7.2; no longer JP1.P1
- net VCC: now also D3.C, K3.2, LED3.A, R28.1, X4.3, X5.3, X6.3
Routing:
- net A2: track 0.00 -> 111.3 mm, vias 0 -> 4
- net RD+: track 140.1 -> 31.6 mm, vias 5 -> 3
- net A3: track 0.00 -> 80.0 mm, vias 0 -> 3
- net D0: track 0.00 -> 58.7 mm, vias 0 -> 3
- net D2: track 0.00 -> 52.6 mm
- net A1: track 0.00 -> 46.5 mm, vias 0 -> 2
- net D1: track 0.00 -> 42.9 mm, vias 0 -> 1
- net D10: track 0.00 -> 25.6 mm, vias 0 -> 2
- net N$54: track 71.5 -> 50.5 mm, vias 4 -> 2
- net VCC: track 272.6 -> 293.4 mm, vias 13 -> 9
- net GND: track 322.7 -> 340.5 mm, vias 7 -> 5
- net N$29: track 0.00 -> 16.3 mm
- net N$15: track 0.00 -> 16.2 mm
- net N$14: track 0.00 -> 16.2 mm
- net N$16: track 0.00 -> 16.2 mm
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
Commit message: pcb
Parts:
- removed CX5: 100n, resistor:C0805
- moved RUSB 70.3 mm to (73.0, 41.9), turned to 270 degrees
- moved R7 17.3 mm to (74.9, 41.9), turned to 90 degrees
- moved R8 15.8 mm to (67.1, 37.4), turned to 90 degrees
- moved X2 13.9 mm to (15.8, 22.1), turned to 270 degrees
- moved C9 7.10 mm to (42.2, 21.2)
- moved R24 6.48 mm to (39.8, 21.2)
- moved BAT1 6.48 mm to (26.4, 16.2)
- moved R23 5.85 mm to (37.3, 21.2)
- moved R10 2.54 mm to (69.1, 27.6)
- moved R11 1.91 mm to (71.9, 27.6)
- moved R9 1.27 mm to (74.4, 27.6)
- moved CX4 1.02 mm to (22.8, 31.7), turned to 0 degrees
- moved RBS 0.90 mm to (44.5, 21.2), turned to 90 degrees
- moved CX3 0.82 mm to (22.8, 29.2), turned to 0 degrees
Connections:
- removed net DTR: CX5.1
- net N$46: no longer CX5.2
Routing:
- net N$45: track 81.2 -> 4.75 mm
- net D-: track 30.9 -> 59.8 mm
- net N$38: track 22.3 -> 4.37 mm
- net VCC: track 293.4 -> 309.4 mm, vias 9 -> 8
- net D+: track 21.5 -> 36.5 mm, vias 1 -> 3
- net N$30: track 12.9 -> 5.75 mm
- net N$8: track 10.4 -> 3.68 mm, vias 1 -> 0
- net N$36: track 8.19 -> 14.9 mm
- net SDA: track 36.6 -> 42.2 mm
- net N$33: track 15.3 -> 9.68 mm
- net GND: track 340.5 -> 345.2 mm, vias 5 -> 4
- net N$59: track 14.0 -> 17.1 mm
- net N$6: track 14.4 -> 16.9 mm
- net VIN: track 33.7 -> 35.7 mm, vias 3 -> 1
- net N$18: track 14.0 -> 12.2 mm
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
Commit message: pcb
prie pabaigos...
Parts:
- removed CX1, CX2: 18p, resistor:C0805
- removed CX3, CX4: 22p, resistor:C0805
- removed DS1307: DS1307, adafruit:SO08
- removed IC6: ENC28J60, SparkFun-DigitalIC:SSOP28DB
- removed L2: Bead, rcl:R0805
- removed R28: 3k3, rcl:R0805
- added C1: 100u, resistor:E2-5
- added C4, C5: 0.1µ, resistor:C0805
- added C6: 18p, resistor:C0805
- added DS1: DS1307, adafruit:SO08
- added IC1: LM1117-33, SparkFun:SOT223
- added L1: Bead, rcl:R0805
- added X10: 22-23-2031, con-molex:22-23-2031
- C3: value 100u -> 0.1u; device resistor:PANASONIC_D -> rcl:C0805
- C7: value 0.1µ -> 18p
- C8: value 0.1µ -> 22p
- C9: value 0.1u -> 22p; device rcl:C0805 -> resistor:C0805
- IC2: value LM1117-33 -> ENC28J60; device SparkFun:SOT223 -> SparkFun-DigitalIC:SSOP28DB
- R1, R3, R5: value 10k -> 470
- R10: value 1k -> 330
- R11: value 620 -> 3k3
- R12: value 330 -> 620
- R13: value 2k -> 1k
- R14: value 3k3 -> 49
- R15: value 470 -> 49
- R16: value 10k -> 49
- R17, R25: value 3k3 -> 10k
- R18: value 470 -> 47
- R19: value 49 -> 47
- R2, R4, R6: value 10k -> 3k3
- R21: value 49 -> 1k
- R22: value 49 -> 10k
- R26: value 470 -> 10k
- R7, R8: value 47 -> 10k
- R9: value 3k3 -> 2k
- X1: value 25MHz -> 32.768kHz; device SparkFun:HC49US -> crystal:TC26H
- X2: value 32.768kHz -> 25MHz; device crystal:TC26H -> SparkFun:HC49US
- X4: device con-phoenix-254:3POL254 -> con-phoenix-254:2POL254
- X7: value 22-23-2031 -> (none); device con-molex:22-23-2031 -> con-phoenix-254:3POL254
- moved T4 73.6 mm to (97.8, 17.8), turned to 270 degrees
- moved R1 72.4 mm to (95.2, 12.7)
- moved R2 71.6 mm to (92.5, 20.6), turned to 0 degrees
- moved R3 67.6 mm to (82.5, 12.7), turned to 90 degrees
- moved R4 64.5 mm to (80.0, 20.9), turned to 0 degrees
- moved R26 63.1 mm to (14.0, 41.9), turned to 270 degrees
- moved T1 61.4 mm to (29.2, 43.2), turned to 180 degrees
- moved R5 60.8 mm to (69.8, 12.7), turned to 90 degrees
- moved R6 57.1 mm to (67.3, 21.6), turned to 0 degrees
- moved R25 55.2 mm to (16.5, 41.9), turned to 270 degrees
- moved R16 44.0 mm to (52.9, 30.9)
- moved R7 40.8 mm to (39.8, 21.2)
- moved C7 40.7 mm to (45.9, 29.1)
- moved C3 39.8 mm to (42.2, 21.2), flipped to the bottom, turned to 270 degrees
- moved R22 39.2 mm to (24.1, 41.9), turned to 270 degrees
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- renumbered CX6 to C2, RJ45 to RJ1, U$2 to U$1
Connections:
- removed net N$15 (its old number): K3.10, X9.1
- removed net N$28 (its old number): K3.5, K3.6, X9.3
- removed net N$29 (its old number): K3.1, X9.2
- new net +3V3: C1.+, IC1.4, IC2.15, IC2.19, IC2.20, IC2.25, IC2.28
- new net +5V: ATTINY.8, C3.1, D1.C, D2.C, D3.C, DS1.8, IC1.3, K1.2, K2.2, K3.2, LED1.A, LED2.A, R7.2, R8.2, U$1.P$6, X5.3, X6.3, X7.3
- new net N$16: K3.10, X10.1
- new net N$19: K3.5, K3.6, X10.3
- new net N$20: K3.1, X10.2
- new net N$27: LED3.A
- net A1: now also X6.2; no longer X5.2
- net A2: now also R2.2; no longer R17.2
- net A3: now also R4.2; no longer R14.2
- net A6: now also R10.2, R9.1; no longer R12.2, R13.1
- net D+: now also R19.1; no longer R8.1
- net D-: now also R18.1; no longer R7.1
- net D0: now also R6.2; no longer R25.2
- net D1: now also X5.2; no longer X4.2
- net D10: now also R21.2; no longer R1.1, R28.2
- net D11: now also IC2.7; no longer IC6.7
- net D12: now also IC2.6; no longer IC6.6
- net D13: now also IC2.8; no longer IC6.8
- net D2: now also X7.2; no longer X6.2
- net D3: now also R22.2; no longer R2.2
- net D4: now also R23.2; no longer R3.2
- net D5: now also R24.2; no longer R4.2
- net D6: now also R25.2; no longer R5.2
- net D7: now also R26.2; no longer R6.2
- net D8: now also IC2.9; no longer IC6.9
- net GND: now also C1.-, C3.2, C4.1, C5.1, C6.2, C7.2, C9.1, DS1.4, IC1.1, IC2.11, IC2.18, IC2.2, IC2.21, IC2.22, X7.1; no longer C3.-, C7.1, C9.2, CX1.2, CX2.2, CX3.1, CX4.1, DS1307.4, IC2.1, IC6.11, IC6.18, IC6.2, IC6.21, IC6.22, X4.1
- net N$1: now also R11.2, R13.1; no longer R10.1, R9.2
- net N$11: now also D1.A, K1.9, R5.2; no longer D3.A, K3.9, R26.2
- net N$12: now also D3.A, K3.9, R1.2, T4.C; no longer D2.A, K1.9, R18.2, T3.C
- net N$13: now also R2.1, T4.B; no longer R17.1, T3.B
- net N$14: now also X9.1; no longer X7.1
- net N$17: now also R6.1; no longer R25.1
- net N$18: now also R11.1; no longer R9.1
- net N$2: now also D2.A, R3.2, T3.C; no longer D1.A, R15.2, T1.C
- net N$21: now also LED3.C, R1.1; no longer LED1.C, R18.1
- net N$22: now also R22.1; no longer R2.1
- net N$23: now also R25.1; no longer R5.1
- net N$24: now also R24.1; no longer R4.1
- net N$25: now also R23.1; no longer R3.1
- net N$26: now also T1.C; no longer T4.C
- net N$3: now also R4.1, T3.B; no longer R14.1, T1.B
- net N$30: now also DS1.2, X1.1; no longer DS1307.2, X2.1
- net N$31: now also LED1.C, R5.1; no longer LED3.C, R26.1
- net N$32: now also C9.2, X2.1; no longer CX4.2, X3.1
- net N$33: now also C8.2, X2.2; no longer CX3.2, X3.2
- net N$34: now also IC2.27; no longer IC6.27
- net N$36: now also DS1.3; no longer DS1307.3
- net N$37: now also IC2.26; no longer IC6.26
- net N$38: now also R19.2; no longer R8.2
- net N$39: now also IC2.1; no longer IC6.1
- net N$4: now also X9.3; no longer X7.3
- net N$41: now also C6.1, IC2.24, X3.2; no longer CX1.1, IC6.24, X1.2
- net N$42: now also C7.1, IC2.23, X3.1; no longer CX2.1, IC6.23, X1.1
- net N$44: now also R21.1, T1.B; no longer R1.2, T4.B
- net N$45: now also R18.2; no longer R7.2
- net N$46: now also R17.1; no longer R16.1
- net N$5: now also X9.2; no longer X7.2
- net N$54: now also C5.2, R15.1, R16.2; no longer C7.2, R19.2, R20.1
- net N$59: now also IC2.14; no longer IC6.14
- net N$6: now also R12.1, R13.2; no longer R10.2, R11.1
- net N$7: now also R3.1; no longer R15.1
- net N$8: now also DS1.1, X1.2; no longer DS1307.1, X2.2
- net N$9: now also R10.1, R12.2; no longer R11.2, R12.1
- net RD+: now also IC2.13, R15.2; no longer IC6.13, R20.2
- net RD-: now also IC2.12, R16.1; no longer IC6.12, R19.1
- net RESET: now also IC2.10; no longer IC6.10
- net SCL: now also DS1.6, R7.1; no longer DS1307.6, R24.1
- net SDA: now also DS1.5, R8.1; no longer DS1307.5, R23.1
- net TCT: now also C4.2, L1.1, R14.2, R20.1; no longer C8.2, L2.1, R21.2, R22.1
- net TD+: now also IC2.17, R20.2; no longer IC6.17, R22.2
- net TD-: now also IC2.16, R14.1; no longer IC6.16, R21.1
- net V$: now also R26.1; no longer R6.1
- net VCC: now also L1.2, R17.2, R9.2; no longer ATTINY.8, C3.+, C9.1, D1.C, D2.C, D3.C, DS1307.8, IC2.4, IC6.15, IC6.19, IC6.20, IC6.25, IC6.28, K1.2, K2.2, K3.2, L2.2, LED1.A, LED2.A, LED3.A, R13.2, R16.2, R23.2, R24.2, R28.1, U$1.P$6, X4.3, X5.3, X6.3
Routing:
- net +5V: track 0.00 -> 199.8 mm, vias 0 -> 1
- net VCC: track 309.4 -> 163.4 mm, vias 8 -> 4
- net TCT: track 61.4 -> 14.1 mm
- net N$54: track 50.5 -> 4.43 mm, vias 2 -> 0
- net +3V3: track 0.00 -> 35.5 mm, vias 0 -> 1
- net GND: track 345.2 -> 322.9 mm, vias 4 -> 2
- net N$20: track 0.00 -> 16.3 mm
- net N$29 (its old number): track 16.3 -> 0.00 mm
- net N$15 (its old number): track 16.2 -> 0.00 mm
- net N$16: track 0.00 -> 16.2 mm
- net N$46: track 105.9 -> 118.1 mm, vias 4 -> 2
- net SDA: track 42.2 -> 54.1 mm
- net N$28 (its old number): track 10.2 -> 0.00 mm
- net N$19: track 0.00 -> 10.2 mm
- net D-: track 59.8 -> 50.1 mm
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
Commit message: pcb prie pabaigos
Parts:
- added C10, C11, C12, C14, C15, C16: 100n, resistor:C0805
- added X11: (no value), con-phoenix-254:2POL254
- X2: value 25MHz -> 16MHz
- moved USB 55.7 mm to (53.7, -1.93), turned to 0 degrees
- moved RUSB 42.7 mm to (48.9, 8.25), turned to 0 degrees
- moved R18 42.2 mm to (48.9, 6.35), turned to 180 degrees
- moved R19 38.2 mm to (40.6, 11.7)
- moved X5 12.7 mm to (25.4, 1.91)
- moved X6 12.7 mm to (34.3, 1.91)
- moved X7 12.7 mm to (43.2, 1.91)
- moved X4 12.7 mm to (17.8, 1.91)
- moved ATTINY 9.09 mm to (39.8, 7.58)
- moved ISP 0.27 mm to (50.3, 17.0), turned to 270 degrees
- moved R14 0.05 mm to (61.0, 33.2)
- turned C1 to 90 degrees
Connections:
- net +3V3: now also C14.1
- net +5V: now also C11.2, C12.2, C15.1, C16.1, L1.2, X11.2
- net GND: now also C10.2, C11.1, C12.1, C14.2, C15.2, C16.2, X11.1
- net VCC: now also C10.1; no longer L1.2
Routing:
- net GND: track 322.9 -> 407.1 mm, vias 2 -> 8
- net +5V: track 199.8 -> 266.8 mm
- net D-: track 50.1 -> 12.2 mm, vias 3 -> 1
- net D+: track 40.9 -> 5.55 mm
- net VCC: track 163.4 -> 136.9 mm
- net VIN: track 33.7 -> 12.5 mm, vias 1 -> 0
- net D2: track 53.6 -> 41.1 mm
- net N$38: track 3.64 -> 14.4 mm
- net A1: track 55.9 -> 48.7 mm, vias 1 -> 2
- net D13: track 36.6 -> 43.0 mm, vias 2 -> 0
- net D1: track 37.0 -> 31.1 mm
- net SDA: track 54.1 -> 48.4 mm, vias 2 -> 4
- net A3: track 80.0 -> 74.6 mm
- net MOSI: track 9.81 -> 15.2 mm, vias 0 -> 1
- net N$46: track 118.1 -> 112.9 mm, vias 2 -> 1
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- added copper zone on layer 1, net +3V3
- added copper zone on layer 16, net N$10
Other:
- board size 100 x 50 mm -> 100 x 50.2 mm
- board text added: "2014.02"
- board text removed: "(2014.02)"
