File: v.2/kolektorius_v2-1.sch (EAGLE design)
At the start: 82 parts, among them IC2 LM1117-33, IC6 ENC28J60, K1 G5V1, K2 G5V1, K3 G5V1, T1 2N2222, T2 2N2222, T3 2N2222, T4 2N2222, U1 ATMEGA328P, X1 25MHz, X2 32.768kHz, X3 25MHz, X7 22-23-2031, X8 22-23-2031, X9 22-23-2031

Commit message: pcb
Parts:
- removed CX5: 100n, resistor:C-EUC0805
Connections:
- removed net DTR: CX5.1
- net N$46: no longer CX5.2
Changed lines of the file:
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@@
 <setting verticaltext="up"/>
 </settings>
-<grid distance="0.05" unitdist="inch" unit="mm" style="lines" multiple="1" display="yes" altdistance="0.025" altunitdist="inch" altunit="mm"/>
+<grid distance="0.1" unitdist="inch" unit="inch" style="lines" multiple="1" display="no" altdistance="0.01" altunitdist="inch" altunit="inch"/>
 <layers>
 <layer number="1" name="Top" color="4" fill="1" visible="no" active="no"/>
@@
 <part name="GND9" library="SparkFun" deviceset="GND" device=""/>
 <part name="R16" library="rcl" deviceset="R-EU_" device="R0805" value="10k"/>
-<part name="CX5" library="resistor" deviceset="C-EU" device="C0805" value="100n"/>
 <part name="+3V7" library="supply1" deviceset="VCC" device=""/>
 <part name="CX6" library="resistor" deviceset="C-EU" device="C0805" value="100n"/>
@@
 <attribute name="VALUE" x="143.256" y="128.27" size="1.778" layer="96" rot="R180"/>
 </instance>
-<instance part="CX5" gate="G$1" x="151.13" y="127" smashed="yes">
-<attribute name="NAME" x="154.559" y="119.634" size="1.778" layer="95" rot="R90"/>
-<attribute name="VALUE" x="157.099" y="119.634" size="1.778" layer="96" rot="R90"/>
-</instance>
 <instance part="+3V7" gate="VCC" x="146.05" y="140.97"/>
 <instance part="CX6" gate="G$1" x="137.16" y="95.25" smashed="yes">
@@
 <segment>
 <pinref part="U1" gate="G$1" pin="PC6(/RESET)"/>
-<wire x1="162.56" y1="113.03" x2="160.02" y2="113.03" width="0.1524" layer="91"/>
 <pinref part="RESET" gate="S" pin="4"/>
 <wire x1="142.24" y1="113.03" x2="146.05" y2="113.03" width="0.1524" layer="91"/>
 <pinref part="RESET" gate="S" pin="3"/>
-<wire x1="146.05" y1="113.03" x2="151.13" y2="113.03" width="0.1524" layer="91"/>
-<wire x1="151.13" y1="113.03" x2="160.02" y2="113.03" width="0.1524" layer="91"/>
+<wire x1="146.05" y1="113.03" x2="162.56" y2="113.03" width="0.1524" layer="91"/>
 <wire x1="142.24" y1="115.57" x2="142.24" y2="113.03" width="0.1524" layer="91"/>
 <pinref part="R16" gate="G$1" pin="1"/>
 <wire x1="146.05" y1="120.65" x2="146.05" y2="113.03" width="0.1524" layer="91"/>
-<pinref part="CX5" gate="G$1" pin="2"/>
-<wire x1="151.13" y1="121.92" x2="151.13" y2="113.03" width="0.1524" layer="91"/>
 </segment>
 </net>
@@
 </segment>
 </net>
-<net name="DTR" class="0">
-<segment>
-<pinref part="CX5" gate="G$1" pin="1"/>
-<wire x1="151.13" y1="129.54" x2="151.13" y2="138.43" width="0.1524" layer="91"/>
-<label x="151.13" y="134.62" size="1.778" layer="95" rot="R90"/>
-</segment>
-</net>

Commit message: pcb
prie pabaigos...
Parts:
- removed CX2: 18p, resistor:C-EUC0805
- removed CX3, CX4: 22p, resistor:C-EUC0805
- removed IC6: ENC28J60, SparkFun-DigitalIC:ENC28J60
- removed R28: 3k3, rcl:R-EU_R0805
- added C1: 100u, resistor:CPOL-EUE2-5
- added C4, C5: 0.1µ, resistor:C-EUC0805
- added IC1: LM1117-33, SparkFun:V_REG_LM1117SOT223
- added X10: 22-23-2031, con-molex:22-23-2031
- C3: value 100u -> 0.1u; device resistor:CPOL-EUD -> rcl:C-EUC0805
- C7: value 0.1µ -> 18p
- C8: value 0.1µ -> 22p
- C9: value 0.1u -> 22p; device rcl:C-EUC0805 -> resistor:C-EUC0805
- IC2: value LM1117-33 -> ENC28J60; device SparkFun:V_REG_LM1117SOT223 -> SparkFun-DigitalIC:ENC28J60
- R1, R3, R5: value 10k -> 470
- R10: value 1k -> 330
- R11: value 620 -> 3k3
- R12: value 330 -> 620
- R13: value 2k -> 1k
- R14: value 3k3 -> 49
- R15: value 470 -> 49
- R16: value 10k -> 49
- R17, R25: value 3k3 -> 10k
- R18: value 470 -> 47
- R19: value 49 -> 47
- R2, R4, R6: value 10k -> 3k3
- R21: value 49 -> 1k
- R22: value 49 -> 10k
- R26: value 470 -> 10k
- R7, R8: value 47 -> 10k
- R9: value 3k3 -> 2k
- X1: value 25MHz -> 32.768kHz; device SparkFun:CRYSTALHC49US -> crystal:CRYSTALTC26H
- X2: value 32.768kHz -> 25MHz; device crystal:CRYSTALTC26H -> SparkFun:CRYSTALHC49US
- X4: device con-phoenix-254:MPT3 -> con-phoenix-254:MPT2; OC_FARNELL (none) -> unknown; OC_NEWARK (none) -> unknown
- X7: value 22-23-2031 -> (none); device con-molex:22-23-2031 -> con-phoenix-254:MPT3
- renumbered CX1 to C6, CX6 to C2, DS1307 to DS1, L2 to L1, RJ45 to RJ1, U$2 to U$1
Connections:
- removed net N$15 (its old number): K32.S, X9-1.S
- removed net N$28 (its old number): K32.P, K32.P@1, X9-3.S
- removed net N$29 (its old number): K32.O, X9-2.S
- new net +3V3: C1.+, IC1.OUT@1, IC2.VDD, IC2.VDDOSC, IC2.VDDPLL, IC2.VDDRX, IC2.VDDTX
- new net +5V: ATTINY.VCC, C3.1, D1.C, D2.C, D3.C, DS1.VCC, IC1.IN, K11.1, K21.1, K31.1, LED1.A, LED2.A, R7.2, R8.2, U$1.VCC, X5-3.1, X6-3.1, X7-3.1
- new net N$16: K32.S, X10-1.S
- new net N$19: K32.P, K32.P@1, X10-3.S
- new net N$20: K32.O, X10-2.S
- new net N$27: LED3.A
- net A1: now also X6-2.1; no longer X5-2.1
- net A2: now also R2.2; no longer R17.2
- net A3: now also R4.2; no longer R14.2
- net A6: now also R10.2, R9.1; no longer R12.2, R13.1
- net D+: now also R19.1; no longer R8.1
- net D-: now also R18.1; no longer R7.1
- net D0: now also R6.2; no longer R25.2
- net D1: now also X5-2.1; no longer X4-2.1
- net D10: now also R21.2; no longer R1.1, R28.2
- net D11: now also IC2.SI; no longer IC6.SI
- net D12: now also IC2.SO; no longer IC6.SO
- net D13: now also IC2.SCK; no longer IC6.SCK
- net D2: now also X7-2.1; no longer X6-2.1
- net D3: now also R22.2; no longer R2.2
- net D4: now also R23.2; no longer R3.2
- net D5: now also R24.2; no longer R4.2
- net D6: now also R25.2; no longer R5.2
- net D7: now also R26.2; no longer R6.2
- net D8: now also IC2.CS; no longer IC6.CS
- net GND: now also C1.-, C3.2, C4.1, C5.1, C7.2, C9.1, IC1.ADJ, IC2.VSS, IC2.VSSOSC, IC2.VSSPLL, IC2.VSSRX, IC2.VSSTX, X7-1.1; no longer C3.-, C7.1, C9.2, CX2.2, CX3.1, CX4.1, IC2.ADJ, IC6.VSS, IC6.VSSOSC, IC6.VSSPLL, IC6.VSSRX, IC6.VSSTX, X4-1.1
- net N$1: now also R11.2, R13.1; no longer R10.1, R9.2
- net N$11: now also D1.A, K11.2, R5.2; no longer D3.A, K31.2, R26.2
- net N$12: now also D3.A, K31.2, R1.2, T4.C; no longer D2.A, K11.2, R18.2, T3.C
- net N$13: now also R2.1, T4.B; no longer R17.1, T3.B
- net N$14: now also X9-1.S; no longer X7-1.S
- net N$17: now also R6.1; no longer R25.1
- net N$18: now also R11.1; no longer R9.1
- net N$2: now also D2.A, R3.2, T3.C; no longer D1.A, R15.2, T1.C
- net N$21: now also LED3.C, R1.1; no longer LED1.C, R18.1
- net N$22: now also R22.1; no longer R2.1
- net N$23: now also R25.1; no longer R5.1
- net N$24: now also R24.1; no longer R4.1
- net N$25: now also R23.1; no longer R3.1
- net N$26: now also T1.C; no longer T4.C
- net N$3: now also R4.1, T3.B; no longer R14.1, T1.B
- net N$30: now also X1.1; no longer X2.1
- net N$31: now also LED1.C, R5.1; no longer LED3.C, R26.1
- net N$32: now also C9.2, X2.1; no longer CX4.2, X3.1
- net N$33: now also C8.2, X2.2; no longer CX3.2, X3.2
- net N$34: now also IC2.LEDA; no longer IC6.LEDA
- net N$37: now also IC2.LEDB; no longer IC6.LEDB
- net N$38: now also R19.2; no longer R8.2
- net N$39: now also IC2.VCAP; no longer IC6.VCAP
- net N$4: now also X9-3.S; no longer X7-3.S
- net N$41: now also IC2.OSC2, X3.2; no longer IC6.OSC2, X1.2
- net N$42: now also C7.1, IC2.OSC1, X3.1; no longer CX2.1, IC6.OSC1, X1.1
- net N$44: now also R21.1, T1.B; no longer R1.2, T4.B
- net N$45: now also R18.2; no longer R7.2
- net N$46: now also R17.1; no longer R16.1
- net N$5: now also X9-2.S; no longer X7-2.S
- net N$54: now also C5.2, R15.1, R16.2; no longer C7.2, R19.2, R20.1
- net N$59: now also IC2.RBIAS; no longer IC6.RBIAS
- net N$6: now also R12.1, R13.2; no longer R10.2, R11.1
- net N$7: now also R3.1; no longer R15.1
- net N$8: now also X1.2; no longer X2.2
- net N$9: now also R10.1, R12.2; no longer R11.2, R12.1
- net RD+: now also IC2.TPIN+, R15.2; no longer IC6.TPIN+, R20.2
- net RD-: now also IC2.TPIN-, R16.1; no longer IC6.TPIN-, R19.1
- net RESET: now also IC2.RESET; no longer IC6.RESET
- net SCL: now also R7.1; no longer R24.1
- net SDA: now also R8.1; no longer R23.1
- net TCT: now also C4.2, R14.2, R20.1; no longer C8.2, R21.2, R22.1
- net TD+: now also IC2.TPOUT+, R20.2; no longer IC6.TPOUT+, R22.2
- net TD-: now also IC2.TPOUT-, R14.1; no longer IC6.TPOUT-, R21.1
- net V$: now also R26.1; no longer R6.1
- net VCC: now also R17.2, R9.2; no longer ATTINY.VCC, C3.+, C9.1, D1.C, D2.C, D3.C, DS1.VCC, IC2.OUT@1, IC6.VDD, IC6.VDDOSC, IC6.VDDPLL, IC6.VDDRX, IC6.VDDTX, K11.1, K21.1, K31.1, LED1.A, LED2.A, LED3.A, R13.2, R16.2, R23.2, R24.2, R28.1, U$1.VCC, X4-3.1, X5-3.1, X6-3.1
Other:
- note removed: "3.3V"
- moved on the sheet: C7, C8, C9, D1, D2, D3, K1, K3, LED1, LED3, R1, R10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

Commit message: pcb prie pabaigos
Parts:
- added C10, C11, C12, C14, C15, C16: 100n, resistor:C-EUC0805
- added X11: (no value), con-phoenix-254:MPT2
- X2: value 25MHz -> 16MHz
Connections:
- net +3V3: now also C14.1
- net +5V: now also C11.2, C12.2, C15.1, C16.1, L1.2, X11-2.1
- net GND: now also C10.2, C11.1, C12.1, C14.2, C15.2, C16.2, X11-1.1
- net VCC: now also C10.1; no longer L1.2
Other:
- moved on the sheet: R18, R19, REA, REB, RUSB, USB
