File: v.2/kolektorius_v2.sch (EAGLE design)
At the start: 73 parts, among them IC2 LM1117-33, IC3 DS1307, IC6 ENC28J60, IC7 ATTINY45SO8S2, K1 G5V1, K2 G5V1, T1 2N2222, T3 2N2222, U1 ATMEGA328P, X1 25MHz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

Commit message: ...
Parts:
- renumbered IC3 to DS1307, IC7 to ATTINY
Connections:
- removed net A4: U1.PC4(ADC4/SDA)
- removed net A5: U1.PC5(ADC5/SCL)
- net SCL: now also U1.PC5(ADC5/SCL)
- net SDA: now also U1.PC4(ADC4/SDA)
Changed lines of the file:
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@@
 <setting verticaltext="up"/>
 </settings>
-<grid distance="1.27" unitdist="mm" unit="mm" style="lines" multiple="1" display="no" altdistance="0.01" altunitdist="inch" altunit="mm"/>
+<grid distance="0.1" unitdist="inch" unit="inch" style="lines" multiple="1" display="no" altdistance="0.01" altunitdist="inch" altunit="inch"/>
 <layers>
 <layer number="1" name="Top" color="4" fill="1" visible="no" active="no"/>
@@
 <part name="GND14" library="SparkFun" deviceset="GND" device=""/>
 <part name="+3V9" library="supply1" deviceset="VCC" device=""/>
-<part name="IC7" library="SparkFun" deviceset="ATTINY45" device="SO8S2"/>
+<part name="ATTINY" library="SparkFun" deviceset="ATTINY45" device="SO8S2"/>
 <part name="RUSB" library="rcl" deviceset="R-EU_" device="R0805" value="1.5k"/>
 <part name="BAT1" library="SparkFunNew" deviceset="BATTERY" device="BATTERY_12MM_SMT"/>
 <part name="REA" library="rcl" deviceset="R-EU_" device="R0805" value="330"/>
 <part name="REB" library="rcl" deviceset="R-EU_" device="R0805" value="330"/>
-<part name="IC3" library="adafruit" deviceset="DS1307" device="SOIC" value="DS1307"/>
+<part name="DS1307" library="adafruit" deviceset="DS1307" device="SOIC" value="DS1307"/>
 <part name="C9" library="rcl" deviceset="C-EU" device="C0805" value="0.1u"/>
 <part name="GND10" library="SparkFun" deviceset="GND" device=""/>
@@
 <instance part="GND14" gate="1" x="120.65" y="13.97"/>
 <instance part="+3V9" gate="VCC" x="116.84" y="77.47"/>
-<instance part="IC7" gate="G$1" x="135.89" y="25.4"/>
+<instance part="ATTINY" gate="G$1" x="135.89" y="25.4"/>
 <instance part="RUSB" gate="G$1" x="116.84" y="69.85" smashed="yes" rot="R90">
 <attribute name="NAME" x="115.316" y="70.1294" size="1.778" layer="95" rot="R180"/>
@@
 <attribute name="VALUE" x="227.33" y="193.802" size="1.778" layer="96" rot="MR180"/>
 </instance>
-<instance part="IC3" gate="G$1" x="85.09" y="102.87" smashed="yes">
+<instance part="DS1307" gate="G$1" x="85.09" y="102.87" smashed="yes">
 <attribute name="NAME" x="72.39" y="90.17" size="1.778" layer="95"/>
 </instance>
@@
 <segment>
 <wire x1="120.65" y1="16.51" x2="120.65" y2="20.32" width="0.1524" layer="91"/>
-<pinref part="IC7" gate="G$1" pin="GND"/>
+<pinref part="ATTINY" gate="G$1" pin="GND"/>
 <pinref part="GND14" gate="1" pin="GND"/>
 </segment>
@@
 <wire x1="100.33" y1="87.63" x2="100.33" y2="90.17" width="0.1524" layer="91"/>
 <junction x="85.09" y="87.63"/>
-<pinref part="IC3" gate="G$1" pin="GND"/>
+<pinref part="DS1307" gate="G$1" pin="GND"/>
 <pinref part="GND6" gate="1" pin="GND"/>
 <pinref part="BAT1" gate="G$1" pin="-"/>
@@
 <wire x1="148.59" y1="27.94" x2="154.94" y2="27.94" width="0.1524" layer="91"/>
 <label x="148.59" y="27.94" size="1.778" layer="95"/>
-<pinref part="IC7" gate="G$1" pin="PB2(SCK/ADC1)"/>
+<pinref part="ATTINY" gate="G$1" pin="PB2(SCK/ADC1)"/>
 </segment>
 <segment>
@@
 <wire x1="148.59" y1="30.48" x2="154.94" y2="30.48" width="0.1524" layer="91"/>
 <label x="148.59" y="30.48" size="1.778" layer="95"/>
-<pinref part="IC7" gate="G$1" pin="PB1(MISO)"/>
+<pinref part="ATTINY" gate="G$1" pin="PB1(MISO)"/>
 </segment>
 <segment>
@@
 <wire x1="148.59" y1="33.02" x2="154.94" y2="33.02" width="0.1524" layer="91"/>
 <label x="148.59" y="33.02" size="1.778" layer="95"/>
-<pinref part="IC7" gate="G$1" pin="PB0(MOSI)"/>
+<pinref part="ATTINY" gate="G$1" pin="PB0(MOSI)"/>
 </segment>
 <segment>
@@
 <segment>
 <wire x1="120.65" y1="36.83" x2="120.65" y2="33.02" width="0.1524" layer="91"/>
-<pinref part="IC7" gate="G$1" pin="VCC"/>
+<pinref part="ATTINY" gate="G$1" pin="VCC"/>
 <pinref part="+3V8" gate="VCC" pin="VCC"/>
 </segment>
@@
 <junction x="60.96" y="128.27"/>
 <label x="55.88" y="128.27" size="1.778" layer="95"/>
-<pinref part="IC3" gate="G$1" pin="VCC"/>
+<pinref part="DS1307" gate="G$1" pin="VCC"/>
 <pinref part="C9" gate="G$1" pin="1"/>
 <pinref part="R23" gate="G$1" pin="2"/>
@@
 <wire x1="66.04" y1="100.33" x2="66.04" y2="107.95" width="0.1524" layer="91"/>
 <label x="55.88" y="100.33" size="1.778" layer="95"/>
-<pinref part="IC3" gate="G$1" pin="SDA"/>
+<pinref part="DS1307" gate="G$1" pin="SDA"/>
 <wire x1="66.04" y1="107.95" x2="66.04" y2="100.33" width="0.1524" layer="91"/>
 <wire x1="66.04" y1="100.33" x2="55.88" y2="100.33" width="0.1524" layer="91"/>
@@
 <junction x="66.04" y="107.95"/>
 </segment>
+<segment>
+<pinref part="U1" gate="G$1" pin="PC4(ADC4/SDA)"/>
+<wire x1="210.82" y1="102.87" x2="215.9" y2="102.87" width="0.1524" layer="91"/>
+<label x="213.36" y="102.87" size="1.778" layer="95"/>
+</segment>
 </net>
 <net name="SCL" class="0">
@@
 <wire x1="69.85" y1="105.41" x2="55.88" y2="105.41" width="0.1524" layer="91"/>
 <label x="55.88" y="105.41" size="1.778" layer="95"/>
-<pinref part="IC3" gate="G$1" pin="SCL"/>
+<pinref part="DS1307" gate="G$1" pin="SCL"/>
 <wire x1="69.85" y1="107.95" x2="69.85" y2="105.41" width="0.1524" layer="91"/>
 <pinref part="R24" gate="G$1" pin="1"/>
 <junction x="69.85" y="107.95"/>
 </segment>
+<segment>
+<pinref part="U1" gate="G$1" pin="PC5(ADC5/SCL)"/>
+<wire x1="210.82" y1="100.33" x2="215.9" y2="100.33" width="0.1524" layer="91"/>
+<label x="213.36" y="100.33" size="1.778" layer="95"/>
+</segment>
 </net>
 <net name="D+" class="0">
@@
 <wire x1="148.59" y1="25.4" x2="154.94" y2="25.4" width="0.1524" layer="91"/>
 <label x="148.59" y="25.4" size="1.778" layer="95"/>
-<pinref part="IC7" gate="G$1" pin="PB3(ADC3)"/>
+<pinref part="ATTINY" gate="G$1" pin="PB3(ADC3)"/>
 </segment>
 <segment>
@@
 <wire x1="148.59" y1="22.86" x2="154.94" y2="22.86" width="0.1524" layer="91"/>
 <label x="148.59" y="22.86" size="1.778" layer="95"/>
-<pinref part="IC7" gate="G$1" pin="PB4(ADC2)"/>
+<pinref part="ATTINY" gate="G$1" pin="PB4(ADC2)"/>
 </segment>
 <segment>
@@
 <net name="N$36" class="0">
 <segment>
-<pinref part="IC3" gate="G$1" pin="VBAT"/>
+<pinref part="DS1307" gate="G$1" pin="VBAT"/>
 <pinref part="BAT1" gate="G$1" pin="+"/>
 </segment>
@@
 <wire x1="173.99" y1="27.94" x2="173.99" y2="20.32" width="0.1524" layer="91"/>
 <wire x1="148.59" y1="20.32" x2="173.99" y2="20.32" width="0.1524" layer="91"/>
-<pinref part="IC7" gate="G$1" pin="PB5(NRES)"/>
+<pinref part="ATTINY" gate="G$1" pin="PB5(NRES)"/>
 <pinref part="SJ1" gate="1" pin="1"/>
 <junction x="173.99" y="20.32"/>
@@
 <segment>
 <pinref part="X2" gate="G$1" pin="2"/>
-<pinref part="IC3" gate="G$1" pin="X1"/>
+<pinref part="DS1307" gate="G$1" pin="X1"/>
 <wire x1="80.01" y1="123.19" x2="80.01" y2="120.65" width="0.1524" layer="91"/>
 </segment>
@@
 <segment>
 <pinref part="X2" gate="G$1" pin="1"/>
-<pinref part="IC3" gate="G$1" pin="X2"/>
+<pinref part="DS1307" gate="G$1" pin="X2"/>
 <wire x1="85.09" y1="123.19" x2="85.09" y2="120.65" width="0.1524" layer="91"/>
 </segment>
@@
 </segment>
 </net>
-<net name="A4" class="0">
-<segment>
-<pinref part="U1" gate="G$1" pin="PC4(ADC4/SDA)"/>
-<wire x1="210.82" y1="102.87" x2="215.9" y2="102.87" width="0.1524" layer="91"/>
-<label x="213.36" y="102.87" size="1.778" layer="95"/>
-</segment>
-</net>
-<net name="A5" class="0">
-<segment>
-<pinref part="U1" gate="G$1" pin="PC5(ADC5/SCL)"/>
-<wire x1="210.82" y1="100.33" x2="215.9" y2="100.33" width="0.1524" layer="91"/>
-<label x="213.36" y="100.33" size="1.778" layer="95"/>
-</segment>
-</net>

Commit message: pcb...
Parts:
- CX3, CX4: value 18p -> 22p
Other:
- moved on the sheet: CX1, CX2, RBS
Changed lines of the file:
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@@
 <part name="R8" library="rcl" deviceset="R-EU_" device="R0805" value="47"/>
 <part name="X3" library="SparkFun" deviceset="CRYSTAL" device="HC49US" value="25MHz"/>
-<part name="CX3" library="resistor" deviceset="C-EU" device="C0805" value="18p"/>
-<part name="CX4" library="resistor" deviceset="C-EU" device="C0805" value="18p"/>
+<part name="CX3" library="resistor" deviceset="C-EU" device="C0805" value="22p"/>
+<part name="CX4" library="resistor" deviceset="C-EU" device="C0805" value="22p"/>
 <part name="GND3" library="SparkFun" deviceset="GND" device=""/>
 <part name="R9" library="rcl" deviceset="R-EU_" device="R0805" value="3k3"/>
@@
 <instance part="L2" gate="G$1" x="276.86" y="180.34" rot="R180"/>
 <instance part="+3V4" gate="VCC" x="179.07" y="208.28"/>
-<instance part="RBS" gate="G$1" x="176.53" y="165.1" smashed="yes" rot="MR180">
-<attribute name="NAME" x="173.99" y="169.1386" size="1.778" layer="95" rot="MR0"/>
-<attribute name="VALUE" x="173.99" y="166.878" size="1.778" layer="96" rot="MR0"/>
+<instance part="RBS" gate="G$1" x="166.37" y="165.1" smashed="yes" rot="MR180">
+<attribute name="NAME" x="168.91" y="169.1386" size="1.778" layer="95" rot="MR0"/>
+<attribute name="VALUE" x="171.45" y="166.878" size="1.778" layer="96" rot="MR0"/>
 </instance>
 <instance part="C8" gate="G$1" x="281.94" y="208.28" smashed="yes">
@@
 </instance>
 <instance part="+3V6" gate="VCC" x="262.89" y="182.88"/>
-<instance part="CX1" gate="G$1" x="168.91" y="189.23" smashed="yes" rot="R270">
-<attribute name="NAME" x="161.544" y="193.421" size="1.778" layer="95"/>
-<attribute name="VALUE" x="161.544" y="190.881" size="1.778" layer="96"/>
-</instance>
-<instance part="CX2" gate="G$1" x="168.91" y="184.15" smashed="yes" rot="R270">
-<attribute name="NAME" x="161.544" y="180.721" size="1.778" layer="95"/>
-<attribute name="VALUE" x="161.544" y="178.181" size="1.778" layer="96"/>
+<instance part="CX1" gate="G$1" x="166.37" y="189.23" smashed="yes" rot="R270">
+<attribute name="NAME" x="166.624" y="193.421" size="1.778" layer="95"/>
+<attribute name="VALUE" x="166.624" y="190.881" size="1.778" layer="96"/>
+</instance>
+<instance part="CX2" gate="G$1" x="166.37" y="184.15" smashed="yes" rot="R270">
+<attribute name="NAME" x="166.624" y="180.721" size="1.778" layer="95"/>
+<attribute name="VALUE" x="166.624" y="178.181" size="1.778" layer="96"/>
 </instance>
 <instance part="GND6" gate="1" x="85.09" y="85.09"/>
@@
 <instance part="X3" gate="G$1" x="156.21" y="85.09" smashed="yes" rot="R90"/>
 <instance part="CX3" gate="G$1" x="148.59" y="87.63" smashed="yes" rot="R90">
-<attribute name="NAME" x="155.956" y="91.059" size="1.778" layer="95" rot="R180"/>
-<attribute name="VALUE" x="155.956" y="93.599" size="1.778" layer="96" rot="R180"/>
+<attribute name="NAME" x="150.876" y="91.059" size="1.778" layer="95" rot="R180"/>
+<attribute name="VALUE" x="155.956" y="91.059" size="1.778" layer="96" rot="R180"/>
 </instance>
 <instance part="CX4" gate="G$1" x="148.59" y="82.55" smashed="yes" rot="R90">
-<attribute name="NAME" x="155.956" y="85.979" size="1.778" layer="95" rot="R180"/>
-<attribute name="VALUE" x="155.956" y="88.519" size="1.778" layer="96" rot="R180"/>
+<attribute name="NAME" x="146.304" y="79.121" size="1.778" layer="95"/>
+<attribute name="VALUE" x="151.384" y="79.121" size="1.778" layer="96"/>
 </instance>
 <instance part="GND3" gate="1" x="144.78" y="77.47"/>
@@
 <wire x1="175.26" y1="154.94" x2="177.8" y2="154.94" width="0.1524" layer="91"/>
 <wire x1="177.8" y1="154.94" x2="181.61" y2="154.94" width="0.1524" layer="91"/>
-<wire x1="171.45" y1="165.1" x2="171.45" y2="154.94" width="0.1524" layer="91"/>
-<wire x1="171.45" y1="154.94" x2="175.26" y2="154.94" width="0.1524" layer="91"/>
-<wire x1="163.83" y1="189.23" x2="163.83" y2="184.15" width="0.1524" layer="91"/>
-<wire x1="163.83" y1="184.15" x2="163.83" y2="154.94" width="0.1524" layer="91"/>
-<wire x1="163.83" y1="154.94" x2="171.45" y2="154.94" width="0.1524" layer="91"/>
+<wire x1="161.29" y1="165.1" x2="161.29" y2="154.94" width="0.1524" layer="91"/>
+<wire x1="161.29" y1="154.94" x2="175.26" y2="154.94" width="0.1524" layer="91"/>
+<wire x1="161.29" y1="189.23" x2="161.29" y2="184.15" width="0.1524" layer="91"/>
+<wire x1="161.29" y1="184.15" x2="161.29" y2="154.94" width="0.1524" layer="91"/>
 <junction x="181.61" y="154.94"/>
 <junction x="181.61" y="152.4"/>
 <junction x="181.61" y="149.86"/>
 <junction x="175.26" y="154.94"/>
-<junction x="163.83" y="184.15"/>
-<junction x="171.45" y="154.94"/>
+<junction x="161.29" y="184.15"/>
+<junction x="161.29" y="154.94"/>
 <junction x="177.8" y="154.94"/>
 <pinref part="IC6" gate="G$1" pin="VSS"/>
@@
 <pinref part="IC6" gate="G$1" pin="RBIAS"/>
 <pinref part="RBS" gate="G$1" pin="2"/>
+<wire x1="171.45" y1="165.1" x2="181.61" y2="165.1" width="0.1524" layer="91"/>
 </segment>
 </net>
 <net name="N$41" class="0">
 <segment>
-<wire x1="171.45" y1="189.23" x2="175.26" y2="189.23" width="0.1524" layer="91"/>
+<wire x1="168.91" y1="189.23" x2="175.26" y2="189.23" width="0.1524" layer="91"/>
 <wire x1="175.26" y1="189.23" x2="175.26" y2="187.96" width="0.1524" layer="91"/>
 <wire x1="175.26" y1="187.96" x2="181.61" y2="187.96" width="0.1524" layer="91"/>
@@
 <pinref part="IC6" gate="G$1" pin="OSC2"/>
 <pinref part="X1" gate="G$1" pin="2"/>
-<junction x="171.45" y="189.23"/>
+<junction x="168.91" y="189.23"/>
+<wire x1="168.91" y1="189.23" x2="171.45" y2="189.23" width="0.1524" layer="91"/>
 </segment>
 </net>
 <net name="N$42" class="0">
 <segment>
-<wire x1="171.45" y1="184.15" x2="175.26" y2="184.15" width="0.1524" layer="91"/>
+<wire x1="168.91" y1="184.15" x2="175.26" y2="184.15" width="0.1524" layer="91"/>
 <wire x1="175.26" y1="185.42" x2="181.61" y2="185.42" width="0.1524" layer="91"/>
 <wire x1="175.26" y1="184.15" x2="175.26" y2="185.42" width="0.1524" layer="91"/>
@@
 <pinref part="IC6" gate="G$1" pin="OSC1"/>
 <pinref part="X1" gate="G$1" pin="1"/>
-<junction x="171.45" y="184.15"/>
-</segment>
-</net>
+<junction x="168.91" y="184.15"/>
+<wire x1="168.91" y1="184.15" x2="171.45" y2="184.15" width="0.1524" layer="91"/>
+</segment>
+</net>

Commit message: pcb
Parts:
- removed JP1, JP3: M022.54MM_SCREWTERM, SparkFun-Connectors:M022.54MM_SCREWTERM
- added D3: (no value), adafruit:DIODEDO-1N4148
- added K3: G5V1, relay:G5V1
- added LED3: (no value), adafruit:LEDSMT1206
- added R25, R28: 3k3, rcl:R-EU_R0805
- added R26: 470, rcl:R-EU_R0805
- added T2, T4: 2N2222, adafruit:2N2222
- added X7, X8, X9: 22-23-2031, con-molex:22-23-2031
Connections:
- removed net N$10: R14.2
- removed net N$27: R17.2
- removed net N$51: R1.2
- new net D0: R25.2, U1.PD0(RXD)
- new net D1: U1.PD1(TXD), X4-2.1
- new net D2: U1.PD2(INT0), X6-2.1
- new net N$11: D3.A, K31.2, R26.2, T2.C
- new net N$17: R25.1, T2.B
- new net N$28: K32.P, K32.P@1, X9-3.S
- new net N$29: K32.O, X9-2.S
- new net N$31: LED3.C, R26.1
- new net N$44: R1.2, T4.B
- net A1: now also X5-2.1
- net A2: now also R17.2
- net A3: now also R14.2
- net D10: now also R1.1, R28.2
- net GND: now also T2.E, T4.E, X4-1.1, X5-1.1, X6-1.1
- net N$14: now also K22.S, X7-1.S; no longer U1.PD0(RXD)
- net N$15: now also K32.S, X9-1.S; no longer U1.PD1(TXD)
- net N$16: now also K12.S, X8-1.S; no longer U1.PD2(INT0)
- net N$19: now also X8-3.S; no longer JP3.2
- net N$20: now also X8-2.S; no longer JP3.1
- net N$26: now also T4.C; no longer R1.1
- net N$4: now also X7-3.S; no longer JP1.2
- net N$5: now also X7-2.S; no longer JP1.1
- net VCC: now also D3.C, K31.1, LED3.A, R28.1, X4-3.1, X5-3.1, X6-3.1
Other:
- moved on the sheet: D2, K1, LED1, R1, R17, R18, T3, X4-1, X4-2, X4-3, X5-1, X5-2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

Commit message: pcb
Parts:
- removed CX5: 100n, resistor:C-EUC0805
Connections:
- removed net DTR: CX5.1
- net N$46: no longer CX5.2
Changed lines of the file:
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@@
 <setting verticaltext="up"/>
 </settings>
-<grid distance="0.05" unitdist="inch" unit="mm" style="lines" multiple="1" display="yes" altdistance="0.025" altunitdist="inch" altunit="mm"/>
+<grid distance="0.635" unitdist="mm" unit="mm" style="lines" multiple="1" display="no" altdistance="0.025" altunitdist="inch" altunit="mm"/>
 <layers>
 <layer number="1" name="Top" color="4" fill="1" visible="no" active="no"/>
@@
 <clearance class="1" value="0.2032"/>
 </class>
+<class number="2" name="GND" width="0.6096" drill="0">
+</class>
+<class number="3" name="signal" width="0.4572" drill="0">
+</class>
 </classes>
 <parts>
@@
 <part name="GND9" library="SparkFun" deviceset="GND" device=""/>
 <part name="R16" library="rcl" deviceset="R-EU_" device="R0805" value="10k"/>
-<part name="CX5" library="resistor" deviceset="C-EU" device="C0805" value="100n"/>
 <part name="+3V7" library="supply1" deviceset="VCC" device=""/>
 <part name="CX6" library="resistor" deviceset="C-EU" device="C0805" value="100n"/>
@@
 <attribute name="VALUE" x="143.256" y="128.27" size="1.778" layer="96" rot="R180"/>
 </instance>
-<instance part="CX5" gate="G$1" x="151.13" y="127" smashed="yes">
-<attribute name="NAME" x="154.559" y="119.634" size="1.778" layer="95" rot="R90"/>
-<attribute name="VALUE" x="157.099" y="119.634" size="1.778" layer="96" rot="R90"/>
-</instance>
 <instance part="+3V7" gate="VCC" x="146.05" y="140.97"/>
 <instance part="CX6" gate="G$1" x="137.16" y="95.25" smashed="yes">
@@
 <instance part="X6" gate="-3" x="293.37" y="74.93"/>
 <instance part="R19" gate="G$1" x="254" y="199.39" smashed="yes">
-<attribute name="NAME" x="251.714" y="198.8566" size="1.1" layer="95"/>
-<attribute name="VALUE" x="251.714" y="200.406" size="0.8" layer="96"/>
+<attribute name="NAME" x="251.714" y="196.3166" size="1.778" layer="95"/>
+<attribute name="VALUE" x="251.714" y="200.406" size="1.778" layer="96"/>
 </instance>
 <instance part="R20" gate="G$1" x="264.16" y="199.39" smashed="yes">
-<attribute name="NAME" x="261.874" y="198.8566" size="1.1" layer="95"/>
-<attribute name="VALUE" x="261.874" y="200.406" size="0.8" layer="96"/>
+<attribute name="NAME" x="261.874" y="196.3166" size="1.778" layer="95"/>
+<attribute name="VALUE" x="261.874" y="200.406" size="1.778" layer="96"/>
 </instance>
 <instance part="R21" gate="G$1" x="276.86" y="199.39" smashed="yes">
-<attribute name="NAME" x="274.574" y="198.8566" size="1.1" layer="95"/>
-<attribute name="VALUE" x="274.574" y="200.406" size="0.8" layer="96"/>
+<attribute name="NAME" x="274.574" y="196.3166" size="1.778" layer="95"/>
+<attribute name="VALUE" x="274.574" y="200.406" size="1.778" layer="96"/>
 </instance>
 <instance part="R22" gate="G$1" x="287.02" y="199.39" smashed="yes">
-<attribute name="NAME" x="284.734" y="198.8566" size="1.1" layer="95"/>
-<attribute name="VALUE" x="284.734" y="200.406" size="0.8" layer="96"/>
+<attribute name="NAME" x="284.734" y="196.3166" size="1.778" layer="95"/>
+<attribute name="VALUE" x="284.734" y="200.406" size="1.778" layer="96"/>
 </instance>
 <instance part="R23" gate="G$1" x="66.04" y="113.03" smashed="yes" rot="R90">
@@
 <segment>
 <pinref part="U1" gate="G$1" pin="PC6(/RESET)"/>
-<wire x1="162.56" y1="113.03" x2="160.02" y2="113.03" width="0.1524" layer="91"/>
 <pinref part="RESET" gate="S" pin="4"/>
 <wire x1="142.24" y1="113.03" x2="146.05" y2="113.03" width="0.1524" layer="91"/>
 <pinref part="RESET" gate="S" pin="3"/>
-<wire x1="146.05" y1="113.03" x2="151.13" y2="113.03" width="0.1524" layer="91"/>
-<wire x1="151.13" y1="113.03" x2="160.02" y2="113.03" width="0.1524" layer="91"/>
+<wire x1="146.05" y1="113.03" x2="162.56" y2="113.03" width="0.1524" layer="91"/>
 <wire x1="142.24" y1="115.57" x2="142.24" y2="113.03" width="0.1524" layer="91"/>
 <pinref part="R16" gate="G$1" pin="1"/>
 <wire x1="146.05" y1="120.65" x2="146.05" y2="113.03" width="0.1524" layer="91"/>
-<pinref part="CX5" gate="G$1" pin="2"/>
-<wire x1="151.13" y1="121.92" x2="151.13" y2="113.03" width="0.1524" layer="91"/>
 </segment>
 </net>
@@
 </segment>
 </net>
-<net name="DTR" class="0">
-<segment>
-<pinref part="CX5" gate="G$1" pin="1"/>
-<wire x1="151.13" y1="129.54" x2="151.13" y2="138.43" width="0.1524" layer="91"/>
-<label x="151.13" y="134.62" size="1.778" layer="95" rot="R90"/>
-</segment>
-</net>
 <net name="N$12" class="0">
 <segment>
@@
 </segment>
 </net>
-<net name="N$26" class="0">
+<net name="N$26" class="3">
 <segment>
 <pinref part="T4" gate="G$1" pin="C"/>
