File: v.2/kolektorius_v2-poligonas.brd (EAGLE design)
At the start: 100 x 50.2 mm, 88 parts, among them IC1 LM1117-33, IC2 ENC28J60, K1 G5V1, K2 G5V1, K3 G5V1, T1 2N2222, T2 2N2222, T3 2N2222, T4 2N2222, U1 ATMEGA328P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

Commit message: pabaiga
Parts:
- X2: value 25MHz -> 16MHz
- moved R17 30.5 mm to (66.0, 35.6)
- moved RESET 21.7 mm to (70.5, 41.0)
- moved X11 3.81 mm to (8.26, 1.91)
- moved C15 1.97 mm to (32.2, 9.40)
Routing:
- net N$46: track 112.9 -> 76.4 mm, vias 1 -> 2
- net +5V: track 267.5 -> 251.4 mm, vias 1 -> 2
- net GND: track 409.1 -> 403.4 mm, vias 8 -> 6
- net A6: track 113.7 -> 118.2 mm
- net VCC: track 136.9 -> 138.2 mm
- net A1: vias 1 -> 2
- added copper zone on layer 16, net N$10
Other:
- board text added: "2014.02"
- board text removed: "(2014.02)"
