File: v1.21_hardware/Order#100038794_2Layer_Green_1.6mm_HASL_5cm_x_5cm.brd (EAGLE design)
At the start: 49.5 x 50 mm, 27 parts, among them J1 POWER, T1 BC337, X1 VCC D2 GND, X2 VCC D8 GND, X3 VCC A3 GND, X4 GND A5 A4 VCC, X5 VCC A2 A1 GND

Commit message: gerber failai i6siuntimui
Parts:
- JP2: value A0 A6 +5V -> +5V A6 A0
- S1: value Right -> (none)
- S2: value Up -> (none)
- S3: value Down -> (none)
- S4: value Left -> (none)
- S5: value Select -> (none)
Connections:
- removed net D0: U$2.D1/TX
- removed net D1: U$2.D0/RX
- removed net N$7: U$2.AREF
Other:
- board text added: "ORDER #100038794"
- board text removed: "ORDER #100022604"
