File: v1.21_hardware/Order#100038794_2Layer_Green_1.6mm_HASL_5cm_x_5cm.sch (EAGLE design)
At the start: 27 parts, among them J1 POWER, T1 BC337, X1 VCC D2 GND, X2 VCC D9 GND, X3 VCC A3 GND, X4 GND A5 A4 VCC, X5 VCC A2 A1 GND

Commit message: gerber failai i6siuntimui
Parts:
- removed JP1: A6 A7, SparkFun:M02PTH
- added JP2: +5V A6 A0, SparkFun-Connectors:M03PTH
- S1: value Right -> (none)
- S2: value Up -> (none)
- S3: value Down -> (none)
- S4: value Left -> (none)
- S5: value Select -> (none)
- X2: value VCC D9 GND -> VCC D8 GND
Connections:
- removed net D0: U$2.D1/TX
- removed net D1: U$2.D0/RX
- removed net N$7: U$2.AREF
- net A0: now also JP2.3; no longer R10.1, R9.2, S1.S, S1.S1
- net A6: now also JP2.2; no longer JP1.1
- net A7: now also R10.1, R9.2, S1.S, S1.S1; no longer JP1.2
- net D8: now also R3.2, X2-2.S; no longer R1.2
- net D9: now also R1.2; no longer R3.2, X2-2.S
- net VCC: now also JP2.1
Other:
- moved on the sheet: R3, R4
