File: v.2.3/kolektorius_v2.2_ch340g.brd (EAGLE design)
At the start: 100 x 50.2 mm, 88 parts, among them IC1 LM1117-33, IC2 ENC28J60, K2 G5V1, K3 JRC-21F(4100), T1 2N2222, T2 2N2222, T3 2N2222, T4 2N2222, U1 ATMEGA328P, X1 32.768kHz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

Commit message: 1.3 versija
programa su 3 klavisais
Parts:
- added C15: 22p, resistor:C0805
- C13: value 0.1u -> 22p; device rcl:C0805 -> resistor:C0805
- X12: value 12MHZ -> 16MHz; device adafruit:CERM_OSC -> SparkFun:HC49US
- moved L1 4.02 mm to (61.6, 27.9)
- moved C4 4.02 mm to (61.5, 30.1)
- moved R15 2.54 mm to (57.4, 30.9)
- moved C13 1.27 mm to (43.2, 8.89)
- moved C5 1.27 mm to (51.8, 30.9)
- moved R16 1.27 mm to (54.1, 30.9)
- moved X12 1.27 mm to (44.5, 14.0), turned to 270 degrees
- moved R10 1.27 mm to (85.9, 35.8), turned to 90 degrees
- turned RIGHT to 270 degrees
Connections:
- removed net N$38: U$2.8, X12.P$3
- net GND: now also C15.1; no longer X12.P$2
- net N$10: now also C13.2, X12.2; no longer X12.P$1
- net N$40: now also C15.2, U$2.8, X12.1; no longer C13.2, U$2.4
Routing:
- net GND: track 0.00 -> 402.0 mm, vias 0 -> 9
- net +5V: track 0.00 -> 303.0 mm, vias 0 -> 5
- net A6: track 0.00 -> 116.2 mm
- net N$46: track 0.00 -> 110.7 mm, vias 0 -> 1
- net A2: track 0.00 -> 93.5 mm, vias 0 -> 5
- net D9: track 0.00 -> 93.3 mm, vias 0 -> 4
- net SDA: track 0.00 -> 82.3 mm, vias 0 -> 2
- net A3: track 0.00 -> 75.2 mm, vias 0 -> 5
- net D12: track 0.00 -> 68.7 mm, vias 0 -> 1
- net SCL: track 0.00 -> 65.6 mm, vias 0 -> 1
- net D11: track 0.00 -> 63.2 mm, vias 0 -> 2
- net A1: track 0.00 -> 58.1 mm, vias 0 -> 2
- net D2: track 0.00 -> 56.1 mm
- net RD+: track 0.00 -> 50.9 mm
- net A0: track 0.00 -> 42.4 mm, vias 0 -> 2
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