File: v.2.3/kolektorius_v2.2_ch340g.sch (EAGLE design)
At the start: 88 parts, among them IC1 LM1117-33, IC2 ENC28J60, K2 G5V1, K3 JRC-21F(4100), T1 2N2222, T2 2N2222, T3 2N2222, T4 2N2222, U1 ATMEGA328P, X1 32.768kHz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

Commit message: 1.3 versija
programa su 3 klavisais
Parts:
- added C15: 22p, resistor:C-EUC0805
- C13: value 0.1u -> 22p; device rcl:C-EUC0805 -> resistor:C-EUC0805
- X12: value 12MHZ -> 16MHz; device adafruit:CERMOSCILL-THM -> SparkFun:CRYSTALHC49US
Connections:
- removed net N$38: U$2.X0, X12.OUT
- net GND: now also C15.1; no longer X12.GND
- net N$10: now also C13.2, X12.2; no longer X12.IN
- net N$40: now also C15.2, U$2.X0, X12.1; no longer C13.2, U$2.V3
Other:
- moved on the sheet: C13
Changed lines of the file:
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@@
 <setting verticaltext="up"/>
 </settings>
-<grid distance="0.1" unitdist="inch" unit="inch" style="lines" multiple="1" display="no" altdistance="0.01" altunitdist="inch" altunit="inch"/>
+<grid distance="1.27" unitdist="mm" unit="mm" style="lines" multiple="1" display="no" altdistance="0.01" altunitdist="inch" altunit="mm"/>
 <layers>
 <layer number="1" name="Top" color="4" fill="1" visible="no" active="no"/>
@@
 <part name="GND20" library="SparkFun" deviceset="GND" device=""/>
 <part name="U$2" library="ch340" deviceset="CH340G" device=""/>
+<part name="X12" library="SparkFun" deviceset="CRYSTAL" device="HC49US" value="16MHz"/>
+<part name="C13" library="resistor" deviceset="C-EU" device="C0805" value="22p"/>
+<part name="C15" library="resistor" deviceset="C-EU" device="C0805" value="22p"/>
 <part name="C17" library="rcl" deviceset="C-US" device="C0805K"/>
 <part name="+3V8" library="supply1" deviceset="+5V" device=""/>
@@
 <part name="R19" library="rcl" deviceset="R-EU_" device="R0805" value="1k"/>
 <part name="+3V9" library="supply1" deviceset="+5V" device=""/>
-<part name="X12" library="adafruit" deviceset="CERMOSCILL" device="-THM" value="12MHZ"/>
-<part name="C13" library="rcl" deviceset="C-EU" device="C0805" value="0.1u"/>
 </parts>
 <sheets>
@@
 <instance part="GND20" gate="1" x="101.6" y="116.84"/>
 <instance part="U$2" gate="G$1" x="124.46" y="12.7"/>
+<instance part="X12" gate="G$1" x="100.33" y="2.54" smashed="yes" rot="R90"/>
+<instance part="C13" gate="G$1" x="91.44" y="5.08" smashed="yes" rot="R90">
+<attribute name="NAME" x="91.186" y="7.239" size="1.778" layer="95" rot="R180"/>
+<attribute name="VALUE" x="98.806" y="7.239" size="1.778" layer="96" rot="R180"/>
+</instance>
+<instance part="C15" gate="G$1" x="91.44" y="0" smashed="yes" rot="R90">
+<attribute name="NAME" x="91.186" y="2.159" size="1.778" layer="95" rot="R180"/>
+<attribute name="VALUE" x="98.806" y="2.159" size="1.778" layer="96" rot="R180"/>
+</instance>
 <instance part="C17" gate="G$1" x="149.86" y="15.24" rot="R90"/>
 <instance part="+3V8" gate="1" x="104.14" y="-17.78" smashed="yes" rot="R90">
@@
 </instance>
 <instance part="+3V9" gate="1" x="119.38" y="58.42"/>
-<instance part="X12" gate="G$1" x="91.44" y="0" smashed="yes" rot="R270">
-<attribute name="NAME" x="90.17" y="6.35" size="1.778" layer="95"/>
-<attribute name="VALUE" x="86.36" y="-6.35" size="1.778" layer="96"/>
-</instance>
-<instance part="C13" gate="G$1" x="92.71" y="12.7" smashed="yes" rot="R90">
-<attribute name="NAME" x="92.456" y="16.129" size="1.778" layer="95" rot="R180"/>
-<attribute name="VALUE" x="95.504" y="14.351" size="1.778" layer="96"/>
-</instance>
 </instances>
 <busses>
@@
 </segment>
 <segment>
+<pinref part="C13" gate="G$1" pin="1"/>
+<wire x1="88.9" y1="5.08" x2="86.36" y2="5.08" width="0.1524" layer="91"/>
+<wire x1="86.36" y1="5.08" x2="86.36" y2="0" width="0.1524" layer="91"/>
+<pinref part="C15" gate="G$1" pin="1"/>
+<wire x1="86.36" y1="0" x2="86.36" y2="-7.62" width="0.1524" layer="91"/>
+<wire x1="88.9" y1="0" x2="86.36" y2="0" width="0.1524" layer="91"/>
+<junction x="86.36" y="0"/>
 <pinref part="U$2" gate="G$1" pin="GND"/>
 <wire x1="111.76" y1="20.32" x2="86.36" y2="20.32" width="0.1524" layer="91"/>
-<wire x1="86.36" y1="20.32" x2="86.36" y2="12.7" width="0.1524" layer="91"/>
+<wire x1="86.36" y1="20.32" x2="86.36" y2="5.08" width="0.1524" layer="91"/>
 <label x="105.41" y="20.32" size="1.778" layer="95"/>
+<junction x="86.36" y="5.08"/>
 <pinref part="USB" gate="G$1" pin="GND"/>
 <pinref part="USB" gate="G$1" pin="ID"/>
-<wire x1="86.36" y1="12.7" x2="86.36" y2="0" width="0.1524" layer="91"/>
-<wire x1="86.36" y1="0" x2="86.36" y2="-7.62" width="0.1524" layer="91"/>
 <wire x1="114.3" y1="-10.16" x2="114.3" y2="-7.62" width="0.1524" layer="91"/>
 <junction x="114.3" y="-10.16"/>
@@
 <junction x="86.36" y="-7.62"/>
 <junction x="114.3" y="-7.62"/>
-<pinref part="X12" gate="G$1" pin="GND"/>
-<wire x1="88.9" y1="0" x2="86.36" y2="0" width="0.1524" layer="91"/>
-<junction x="86.36" y="0"/>
-<wire x1="91.44" y1="12.7" x2="90.17" y2="12.7" width="0.1524" layer="91"/>
-<junction x="86.36" y="12.7"/>
-<pinref part="C13" gate="G$1" pin="1"/>
-<wire x1="90.17" y1="12.7" x2="86.36" y2="12.7" width="0.1524" layer="91"/>
-<junction x="90.17" y="12.7"/>
 </segment>
 <segment>
@@
 </segment>
 </net>
+<net name="N$10" class="0">
+<segment>
+<pinref part="U$2" gate="G$1" pin="XI"/>
+<pinref part="X12" gate="G$1" pin="2"/>
+<wire x1="111.76" y1="5.08" x2="100.33" y2="5.08" width="0.1524" layer="91"/>
+<pinref part="C13" gate="G$1" pin="2"/>
+<wire x1="100.33" y1="5.08" x2="96.52" y2="5.08" width="0.1524" layer="91"/>
+<junction x="100.33" y="5.08"/>
+</segment>
+</net>
+<net name="N$40" class="0">
+<segment>
+<pinref part="C15" gate="G$1" pin="2"/>
+<pinref part="X12" gate="G$1" pin="1"/>
+<wire x1="96.52" y1="0" x2="100.33" y2="0" width="0.1524" layer="91"/>
+<pinref part="U$2" gate="G$1" pin="X0"/>
+<wire x1="100.33" y1="0" x2="111.76" y2="0" width="0.1524" layer="91"/>
+<wire x1="111.76" y1="0" x2="111.76" y2="2.54" width="0.1524" layer="91"/>
+<junction x="100.33" y="0"/>
+</segment>
+</net>
 <net name="N$43" class="0">
 <segment>
@@
 </segment>
 </net>
-<net name="N$10" class="0">
-<segment>
-<pinref part="U$2" gate="G$1" pin="XI"/>
-<pinref part="X12" gate="G$1" pin="IN"/>
-<wire x1="111.76" y1="5.08" x2="96.52" y2="5.08" width="0.1524" layer="91"/>
-<junction x="96.52" y="5.08"/>
-</segment>
-</net>
-<net name="N$38" class="0">
-<segment>
-<pinref part="U$2" gate="G$1" pin="X0"/>
-<wire x1="111.76" y1="2.54" x2="101.6" y2="2.54" width="0.1524" layer="91"/>
-<wire x1="101.6" y1="2.54" x2="101.6" y2="-5.08" width="0.1524" layer="91"/>
-<pinref part="X12" gate="G$1" pin="OUT"/>
-<wire x1="101.6" y1="-5.08" x2="96.52" y2="-5.08" width="0.1524" layer="91"/>
-<junction x="96.52" y="-5.08"/>
-</segment>
-</net>
-<net name="N$40" class="0">
-<segment>
-<pinref part="U$2" gate="G$1" pin="V3"/>
-<wire x1="111.76" y1="12.7" x2="97.79" y2="12.7" width="0.1524" layer="91"/>
-<pinref part="C13" gate="G$1" pin="2"/>
-<wire x1="97.79" y1="12.7" x2="96.52" y2="12.7" width="0.1524" layer="91"/>
-<junction x="97.79" y="12.7"/>
-</segment>
-</net>
