File: v1.4/v1.4.sch (EAGLE design)
At the start: 55 parts, among them IC1 LM1117-33, T1 2N2222, T2 2N2222, U1 ATMEGA328P, X1 32.768kHz, X11 , X2 16MHz, X3 , X4 , X5 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

Commit message: pakeitimai
Parts:
- removed R1, R2, R3, R4, R5: 10k, rcl:R-EU_R0805
- removed R6: 1k, rcl:R-EU_R0805
- removed T1: 2N2222, adafruit:2N2222
- U$1: value CELLPHONE_NOKIA_5100 -> 1.44"-TFT-V1.1; device DIY-Cellphone:CELLPHONE_NOKIA_5100 -> tft_1.8:1.44"-TFT-V1.1
Connections:
- removed net N$2: R5.2, U$1.CLK'
- removed net N$26: T1.C, U$1.BL'
- removed net N$3: R4.2, U$1.DIN'
- removed net N$4: R3.2, U$1.DC'
- removed net N$44: R6.1, T1.B
- removed net N$5: R2.2, U$1.CE'
- removed net N$6: R1.2, U$1.RST'
- net +3V3: now also U$1.LED, U$1.VCC
- net +5V: no longer U$1.VCC'
- net A0: no longer R5.1
- net D11/MOSI: now also U$1.SDA
- net D13/SCK: now also U$1.SCK
- net D2: no longer SJ1.2, X7-2.1
- net D3: now also U$1.RESET
- net D4: now also U$1.CS; no longer R4.1
- net D5: now also U$1.A0; no longer R3.1
- net D6: no longer R2.1
- net D7: now also SJ1.2, X7-2.1; no longer R1.1
- net D9: no longer R6.2
- net GND: now also U$1.GND; no longer T1.E, U$1.GND'
